File: legoPFremote/legoPFremote/legoPFremote.brd (EAGLE design)
At the start: 130.8 x 78.7 mm, 46 parts, among them IC1 MCP73831/OT, SW1 440BS67082622, SW2 440BS67082622, SW3 440BS67082622, SW4 440BS67082622, U1 3.3V

Commit message: WIP
Parts:
- added U$4, U$5, U$6, U$7: MOUNTINGHOLE3.0THIN, microbuilder:MOUNTINGHOLE_3.0_PLATEDTHIN
- moved U$3 46.9 mm to (25.4, 16.5)
- moved LED1 41.3 mm to (26.7, 31.8)
- moved R3 24.7 mm to (31.8, 17.8)
- moved C8 22.5 mm to (31.8, 20.3)
- moved C4 21.6 mm to (31.8, 22.9)
- moved IC1 20.9 mm to (20.3, 24.6)
- moved RESET 20.7 mm to (73.7, 26.7)
- moved POWER 19.4 mm to (2.54, 20.3), turned to 270 degrees
- moved R13 19.3 mm to (21.2, 30.5)
- moved Q1 19.1 mm to (52.1, 55.9)
- moved R7 17.7 mm to (57.1, 55.9)
- moved R14 16.7 mm to (21.2, 27.9)
- moved LED5 16.5 mm to (47.0, 57.1)
- moved LED6 16.5 mm to (40.6, 57.1)
- moved LED7 16.5 mm to (34.3, 57.1)
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Routing:
- net GND: track 357.1 -> 40.3 mm, vias 4 -> 0
- net N$12: track 169.3 -> 0.00 mm
- net VCC: track 149.5 -> 0.00 mm, vias 3 -> 0
- net +3V3: track 74.6 -> 0.00 mm, vias 4 -> 0
- net +5V: track 88.2 -> 29.5 mm, vias 2 -> 0
- net AREF: track 50.0 -> 0.00 mm, vias 2 -> 0
- net N$9: track 34.9 -> 0.00 mm, vias 1 -> 0
- net RST: track 28.4 -> 0.00 mm
- net SCK: track 27.7 -> 0.00 mm
- net MOSI: track 27.6 -> 0.00 mm, vias 1 -> 0
- net USB_D+: track 27.2 -> 0.00 mm, vias 2 -> 0
- net USB_D-: track 27.5 -> 2.12 mm, vias 2 -> 0
- net MISO: track 23.8 -> 0.00 mm, vias 1 -> 0
- net SDA: track 18.8 -> 0.00 mm, vias 3 -> 0
- net VBAT: track 36.2 -> 21.7 mm, vias 1 -> 0
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Other:
- board size 130.8 x 78.7 mm -> 87.6 x 48.3 mm
