File: legoPFremote/legoPFremote/legoPFremote.sch (EAGLE design)
At the start: 46 parts, among them IC1 MCP73831/OT, SW1 440BS67082622, SW2 440BS67082622, SW3 440BS67082622, SW4 440BS67082622, U1 3.3V

Commit message: WIP
Parts:
- added U$4, U$5, U$6, U$7: MOUNTINGHOLE3.0THIN, microbuilder:MOUNTINGHOLE3.0THIN
Changed lines of the file:
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@@
 <part name="U$3" library="an-erd" deviceset="I2C_OLED_DISPLAY" device=""/>
 <part name="+3V3" library="supply1" library_urn="urn:adsk.eagle:library:371" deviceset="+3V3" device=""/>
+<part name="U$4" library="microbuilder" deviceset="MOUNTINGHOLE" device="3.0THIN"/>
+<part name="U$5" library="microbuilder" deviceset="MOUNTINGHOLE" device="3.0THIN"/>
+<part name="U$6" library="microbuilder" deviceset="MOUNTINGHOLE" device="3.0THIN"/>
+<part name="U$7" library="microbuilder" deviceset="MOUNTINGHOLE" device="3.0THIN"/>
 </parts>
 <sheets>
@@
 <instance part="U$3" gate="G$1" x="106.68" y="114.3"/>
 <instance part="+3V3" gate="G$1" x="203.2" y="177.8"/>
+<instance part="U$4" gate="G$1" x="157.48" y="182.88"/>
+<instance part="U$5" gate="G$1" x="157.48" y="177.8"/>
+<instance part="U$6" gate="G$1" x="157.48" y="172.72"/>
+<instance part="U$7" gate="G$1" x="157.48" y="167.64"/>
 </instances>
 <busses>
