File: POIstick/POIstick.brd (EAGLE design)
At the start: 86 x 22.9 mm, 41 parts, among them SW1 431151015826, SW2 431151015826, U1 CR2032-SNAPDRAGONCR2032, X1 8MHz

Commit message: Rev 2
Parts:
- added AREF: PTR1B1,27, testpad:B1,27
- added C7: 0.1uF, microbuilder:0805
- added SW3: (no value), adafruit:PUSHBUTTON_SMD_SJ
- X1: value 8MHz -> 2MHz
- moved SW1 2.29 mm to (37.5, 76.2)
- moved SW2 2.29 mm to (37.5, 61.0)
Connections:
- new net PB0: SW2.2, U$1.8
- net AREF: now also AREF.TP, C7.1
- net GND: now also C7.2, SW2.1, SW3.P$2; no longer SW2.2
- net PE6: now also SW3.P$1; no longer SW2.1
Routing:
- net PB0: track 0.00 -> 37.3 mm, vias 0 -> 2
- net AREF: track 0.00 -> 30.6 mm, vias 0 -> 2
- net PE6: track 39.3 -> 45.4 mm
- net GND: track 156.9 -> 162.9 mm
- net RST: track 61.8 -> 60.4 mm
- removed copper zone on layer 16, net GND
- removed copper zone on layer 1, net N$32
Other:
- board text added: "ATmega32U4"
- board text added: "CONF"
- board text added: "START!"
- board text removed: "FCT"

Commit message: POIstick Rev 3
Parts:
- removed SW3: (no value), adafruit:PUSHBUTTON_SMD_SJ
- added LED13: APT2012SECK, microbuilder:CHIPLED_0805
- added R15: 47, microbuilder:0805
- added S1: MOMENTARY-SWITCH-SPST-SMD-12MM, SparkFun-Switches:TACTILE_SWITCH_SMD_12MM
- added S3: (no value), SparkFun-Switches:SWITCH_SPST_SMD_A
Connections:
- new net N$32: LED13.C, R15.1
- new net N$33: S3.1, U1.V+
- new net PD5: LED13.A, U$1.22
- net GND: now also R15.2, S1.3; no longer SW3.P$2
- net PE6: now also S1.1; no longer SW3.P$1
- net VCC: now also S3.2; no longer U1.V+
Routing:
- net N$33: track 0.00 -> 31.3 mm
- net VCC: track 129.9 -> 111.5 mm
- net PD5: track 0.00 -> 10.8 mm, vias 0 -> 2
- net PE6: track 45.4 -> 53.4 mm
- net GND: track 162.9 -> 166.9 mm
- net N$32: track 0.00 -> 2.32 mm
- net +3V3: track 9.46 -> 11.0 mm
- net PB0: track 37.3 -> 38.7 mm
- net N$25: track 5.57 -> 6.16 mm
- added copper zone on layer 1, net GND
- added copper zone on layer 16, net GND
Other:
- board text added: "...running!"

Commit message: POIstick Rev 7
Parts:
- PTCFUSE: value 250mA -> 500mA
- moved R3 0.68 mm to (42.8, 73.0)
- moved R4 0.65 mm to (47.6, 73.0)
- moved R10 0.63 mm to (78.0, 73.0)
- moved R11 0.63 mm to (83.1, 73.0)
- moved R12 0.63 mm to (88.1, 73.0)
- moved R13 0.63 mm to (93.2, 73.0)
- moved R14 0.63 mm to (98.3, 73.0)
- moved R5 0.63 mm to (52.6, 73.0)
- moved R6 0.63 mm to (57.7, 73.0)
- moved R7 0.63 mm to (62.7, 73.0)
- moved R8 0.63 mm to (67.8, 73.0)
- moved R9 0.63 mm to (72.9, 73.0)
- moved LED1 0.38 mm to (42.7, 77.5)
- moved LED2 0.13 mm to (47.6, 77.5)
- renumbered F2 to PTCFUSE
Routing:
- net GND: track 166.9 -> 168.4 mm
- net AREF: track 30.6 -> 31.4 mm
- net N$8: track 1.81 -> 2.45 mm
- net N$30: track 1.81 -> 2.45 mm
- net N$28: track 1.81 -> 2.45 mm
- net N$26: track 1.81 -> 2.45 mm
- net N$24: track 1.81 -> 2.45 mm
- net N$22: track 1.81 -> 2.45 mm
- net N$20: track 1.81 -> 2.45 mm
- net N$18: track 1.81 -> 2.45 mm
- net N$16: track 1.81 -> 2.45 mm
- net N$14: track 1.81 -> 2.45 mm
- net N$12: track 1.81 -> 2.45 mm
- net N$10: track 1.81 -> 2.45 mm

Commit message: UCAP 0.1uF, replace 3.3V -> VCC
Parts:
- C8: value 0.1uF -> 1uF
Connections:
- net +3V3 renamed N$34
Changed lines of the file:
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@@
 <element name="R14" library="microbuilder" package="0805" value="47" x="98.298" y="73.025" smashed="yes" rot="MR270"/>
 <element name="U1" library="CR2032-SnapDragon" package="CR2032-SNAPDRAGON" value="CR2032-SNAPDRAGONCR2032" x="30.607" y="68.58" smashed="yes" rot="MR0"/>
-<element name="C8" library="microbuilder" package="0805" value="0.1uF" x="68.58" y="59.69" smashed="yes"/>
+<element name="C8" library="microbuilder" package="0805" value="1uF" x="68.58" y="59.69" smashed="yes"/>
 <element name="C3" library="microbuilder" package="0805" value="0.1uF" x="68.58" y="62.23" smashed="yes"/>
 <element name="C4" library="microbuilder" package="0805" value="0.1uF" x="64.77" y="60.96" smashed="yes"/>
@@
 <wire x1="87.95" y1="68.9" x2="82.55" y2="63.5" width="0.254" layer="1"/>
 </signal>
-<signal name="+3V3">
-<contactref element="U$1" pad="6"/>
-<contactref element="C8" pad="1"/>
-<wire x1="73.368778125" y1="64.478778125" x2="72.39" y2="63.5" width="0.254" layer="1"/>
-<via x="72.39" y="63.5" extent="1-16" drill="0.35"/>
-<wire x1="72.39" y1="63.5" x2="72.39" y2="63.2432" width="0.254" layer="16"/>
-<wire x1="72.39" y1="63.2432" x2="66.421" y2="58.5442" width="0.254" layer="16"/>
-<via x="66.421" y="58.5442" extent="1-16" drill="0.35"/>
-<wire x1="66.421" y1="58.5442" x2="67.691" y2="59.629" width="0.254" layer="1"/>
-<wire x1="67.691" y1="59.629" x2="67.63" y2="59.69" width="0.254" layer="1"/>
-</signal>
 <signal name="AREF">
 <contactref element="U$1" pad="42"/>
@@
 <wire x1="23.114" y1="61.468" x2="16.002" y2="68.58" width="0.508" layer="16"/>
 </signal>
+<signal name="N$34">
+<contactref element="U$1" pad="6"/>
+<contactref element="C8" pad="1"/>
+<wire x1="73.368778125" y1="64.478778125" x2="72.39" y2="63.5" width="0.254" layer="1"/>
+<via x="72.39" y="63.5" extent="1-16" drill="0.35"/>
+<wire x1="72.39" y1="63.5" x2="72.39" y2="63.2432" width="0.254" layer="16"/>
+<wire x1="72.39" y1="63.2432" x2="66.421" y2="58.5442" width="0.254" layer="16"/>
+<via x="66.421" y="58.5442" extent="1-16" drill="0.35"/>
+<wire x1="66.421" y1="58.5442" x2="67.691" y2="59.629" width="0.254" layer="1"/>
+<wire x1="67.691" y1="59.629" x2="67.63" y2="59.69" width="0.254" layer="1"/>
+</signal>
 </signals>
