File: POIstick/POIstick.sch (EAGLE design)
At the start: 41 parts, among them SW1 431151015826, SW2 431151015826, U1 CR2032-SNAPDRAGONCR2032, X1 8MHz

Commit message: Rev 2
Parts:
- added AREF: PTR1B1,27, testpad:PTR1B1,27
- added C7: 0.1uF, microbuilder:CAP_CERAMIC0805
- added SW3: (no value), adafruit:SWITCH_PUSHBUTTONSOFTTOUCHSMD_SJ
- X1: value 8MHz -> 2MHz
Connections:
- new net PB0: SW2.2, U$1.PB0(SS)
- net AREF: now also AREF.TP, C7.P$1
- net GND: now also C7.P$2, SW2.1, SW3.P$2; no longer SW2.2
- net PE6: now also SW3.P$1; no longer SW2.1
Other:
- moved on the sheet: SW2
Changed lines of the file:
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@@
 <grid distance="0.1" unitdist="inch" unit="inch" style="lines" multiple="1" display="no" altdistance="0.01" altunitdist="inch" altunit="inch"/>
 <layers>
-<layer number="1" name="Top" color="4" fill="1" visible="yes" active="no"/>
-<layer number="16" name="Bottom" color="1" fill="1" visible="yes" active="no"/>
-<layer number="17" name="Pads" color="2" fill="1" visible="yes" active="no"/>
-<layer number="18" name="Vias" color="2" fill="1" visible="yes" active="no"/>
-<layer number="19" name="Unrouted" color="6" fill="1" visible="yes" active="no"/>
-<layer number="20" name="Dimension" color="15" fill="1" visible="yes" active="no"/>
-<layer number="21" name="tPlace" color="7" fill="1" visible="yes" active="no"/>
-<layer number="22" name="bPlace" color="7" fill="1" visible="yes" active="no"/>
-<layer number="23" name="tOrigins" color="15" fill="1" visible="yes" active="no"/>
-<layer number="24" name="bOrigins" color="15" fill="1" visible="yes" active="no"/>
-<layer number="25" name="tNames" color="7" fill="1" visible="yes" active="no"/>
-<layer number="26" name="bNames" color="7" fill="1" visible="yes" active="no"/>
-<layer number="27" name="tValues" color="7" fill="1" visible="yes" active="no"/>
-<layer number="28" name="bValues" color="7" fill="1" visible="yes" active="no"/>
+<layer number="1" name="Top" color="4" fill="1" visible="no" active="no"/>
+<layer number="16" name="Bottom" color="1" fill="1" visible="no" active="no"/>
+<layer number="17" name="Pads" color="2" fill="1" visible="no" active="no"/>
+<layer number="18" name="Vias" color="2" fill="1" visible="no" active="no"/>
+<layer number="19" name="Unrouted" color="6" fill="1" visible="no" active="no"/>
+<layer number="20" name="Dimension" color="15" fill="1" visible="no" active="no"/>
+<layer number="21" name="tPlace" color="7" fill="1" visible="no" active="no"/>
+<layer number="22" name="bPlace" color="7" fill="1" visible="no" active="no"/>
+<layer number="23" name="tOrigins" color="15" fill="1" visible="no" active="no"/>
+<layer number="24" name="bOrigins" color="15" fill="1" visible="no" active="no"/>
+<layer number="25" name="tNames" color="7" fill="1" visible="no" active="no"/>
+<layer number="26" name="bNames" color="7" fill="1" visible="no" active="no"/>
+<layer number="27" name="tValues" color="7" fill="1" visible="no" active="no"/>
+<layer number="28" name="bValues" color="7" fill="1" visible="no" active="no"/>
 <layer number="29" name="tStop" color="7" fill="3" visible="no" active="no"/>
 <layer number="30" name="bStop" color="7" fill="6" visible="no" active="no"/>
@@
 <layer number="35" name="tGlue" color="7" fill="4" visible="no" active="no"/>
 <layer number="36" name="bGlue" color="7" fill="5" visible="no" active="no"/>
-<layer number="37" name="tTest" color="7" fill="1" visible="yes" active="no"/>
-<layer number="38" name="bTest" color="7" fill="1" visible="yes" active="no"/>
+<layer number="37" name="tTest" color="7" fill="1" visible="no" active="no"/>
+<layer number="38" name="bTest" color="7" fill="1" visible="no" active="no"/>
 <layer number="39" name="tKeepout" color="4" fill="11" visible="no" active="no"/>
 <layer number="40" name="bKeepout" color="1" fill="11" visible="no" active="no"/>
@@
 <layer number="44" name="Drills" color="7" fill="1" visible="no" active="no"/>
 <layer number="45" name="Holes" color="7" fill="1" visible="no" active="no"/>
-<layer number="46" name="Milling" color="3" fill="1" visible="yes" active="no"/>
-<layer number="47" name="Measures" color="7" fill="1" visible="yes" active="no"/>
-<layer number="48" name="Document" color="7" fill="1" visible="yes" active="no"/>
-<layer number="49" name="Reference" color="7" fill="1" visible="yes" active="no"/>
-<layer number="50" name="dxf" color="7" fill="1" visible="yes" active="no"/>
-<layer number="51" name="tDocu" color="7" fill="1" visible="yes" active="no"/>
-<layer number="52" name="bDocu" color="7" fill="1" visible="yes" active="no"/>
-<layer number="53" name="tGND_GNDA" color="7" fill="9" visible="yes" active="no"/>
-<layer number="54" name="bGND_GNDA" color="1" fill="9" visible="yes" active="no"/>
-<layer number="56" name="wert" color="7" fill="1" visible="yes" active="no"/>
-<layer number="57" name="tCAD" color="7" fill="1" visible="yes" active="no"/>
-<layer number="59" name="tCarbon" color="7" fill="1" visible="yes" active="no"/>
-<layer number="60" name="bCarbon" color="7" fill="1" visible="yes" active="no"/>
+<layer number="46" name="Milling" color="3" fill="1" visible="no" active="no"/>
+<layer number="47" name="Measures" color="7" fill="1" visible="no" active="no"/>
+<layer number="48" name="Document" color="7" fill="1" visible="no" active="no"/>
+<layer number="49" name="Reference" color="7" fill="1" visible="no" active="no"/>
+<layer number="50" name="dxf" color="7" fill="1" visible="no" active="no"/>
+<layer number="51" name="tDocu" color="7" fill="1" visible="no" active="no"/>
+<layer number="52" name="bDocu" color="7" fill="1" visible="no" active="no"/>
+<layer number="53" name="tGND_GNDA" color="7" fill="9" visible="no" active="no"/>
+<layer number="54" name="bGND_GNDA" color="1" fill="9" visible="no" active="no"/>
+<layer number="56" name="wert" color="7" fill="1" visible="no" active="no"/>
+<layer number="57" name="tCAD" color="7" fill="1" visible="no" active="no"/>
+<layer number="59" name="tCarbon" color="7" fill="1" visible="no" active="no"/>
+<layer number="60" name="bCarbon" color="7" fill="1" visible="no" active="no"/>
 <layer number="90" name="Modules" color="5" fill="1" visible="yes" active="yes"/>
 <layer number="91" name="Nets" color="2" fill="1" visible="yes" active="yes"/>
@@
 <part name="GND2" library="supply1" library_urn="urn:adsk.eagle:library:371" deviceset="GND" device=""/>
 <part name="GND3" library="supply1" library_urn="urn:adsk.eagle:library:371" deviceset="GND" device=""/>
-<part name="X1" library="adafruit" deviceset="XTAL" device="NX5032" value="8MHz"/>
+<part name="X1" library="adafruit" deviceset="XTAL" device="NX5032" value="2MHz"/>
 <part name="+3V1" library="supply1" library_urn="urn:adsk.eagle:library:371" deviceset="+3V3" device=""/>
 <part name="GND4" library="supply1" library_urn="urn:adsk.eagle:library:371" deviceset="GND" device=""/>
@@
 <part name="P+4" library="supply1" library_urn="urn:adsk.eagle:library:371" deviceset="VCC" device=""/>
 <part name="SW1" library="Wurth_Elektronik_Electromechanic_Switchs_rev15b" deviceset="431151015826" device=""/>
+<part name="SW3" library="adafruit" library_urn="urn:adsk.eagle:library:420" deviceset="SWITCH_PUSHBUTTON" device="SOFTTOUCHSMD_SJ"/>
 <part name="SW2" library="Wurth_Elektronik_Electromechanic_Switchs_rev15b" deviceset="431151015826" device=""/>
+<part name="C7" library="microbuilder" deviceset="CAP_CERAMIC" device="0805" value="0.1uF"/>
+<part name="GND9" library="supply1" library_urn="urn:adsk.eagle:library:371" deviceset="GND" device=""/>
+<part name="AREF" library="testpad" library_urn="urn:adsk.eagle:library:385" deviceset="PTR1" device="B1,27" package3d_urn="urn:adsk.eagle:package:27944/1" value="PTR1B1,27"/>
 </parts>
 <sheets>
@@
 <instance part="P+4" gate="VCC" x="-35.56" y="35.56"/>
 <instance part="SW1" gate="G$1" x="119.38" y="25.4"/>
-<instance part="SW2" gate="G$1" x="119.38" y="2.54"/>
+<instance part="SW3" gate="G$1" x="119.38" y="7.62"/>
+<instance part="SW2" gate="G$1" x="119.38" y="-7.62" rot="MR0"/>
+<instance part="C7" gate="G$1" x="-7.62" y="15.24"/>
+<instance part="GND9" gate="1" x="-7.62" y="10.16"/>
+<instance part="AREF" gate="G$1" x="-12.7" y="20.32"/>
 </instances>
 <busses>
@@
 </segment>
 <segment>
-<pinref part="SW2" gate="G$1" pin="2"/>
-<wire x1="123.19" y1="7.62" x2="137.16" y2="7.62" width="0.1524" layer="91"/>
 <label x="132.08" y="7.62" size="1.778" layer="95"/>
+<pinref part="SW3" gate="G$1" pin="P$2"/>
+<wire x1="124.46" y1="7.62" x2="137.16" y2="7.62" width="0.1524" layer="91"/>
+</segment>
+<segment>
+<pinref part="SW2" gate="G$1" pin="1"/>
+<wire x1="123.19" y1="-2.54" x2="137.16" y2="-2.54" width="0.1524" layer="91"/>
+<label x="132.08" y="-2.54" size="1.778" layer="95"/>
+</segment>
+<segment>
+<pinref part="C7" gate="G$1" pin="P$2"/>
+<pinref part="GND9" gate="1" pin="GND"/>
 </segment>
 </net>
@@
 <label x="17.78" y="50.8" size="1.778" layer="95"/>
 </segment>
+<segment>
+<pinref part="C7" gate="G$1" pin="P$1"/>
+<wire x1="-7.62" y1="20.32" x2="-7.62" y2="22.86" width="0.1524" layer="91"/>
+<wire x1="-7.62" y1="22.86" x2="2.54" y2="22.86" width="0.1524" layer="91"/>
+<label x="0" y="22.86" size="1.778" layer="95"/>
+<wire x1="-12.7" y1="22.86" x2="-7.62" y2="22.86" width="0.1524" layer="91"/>
+<junction x="-7.62" y="22.86"/>
+<pinref part="AREF" gate="G$1" pin="TP"/>
+</segment>
 </net>
 <net name="MISO" class="0">
@@
 </segment>
 <segment>
-<pinref part="SW2" gate="G$1" pin="1"/>
-<wire x1="115.57" y1="7.62" x2="96.52" y2="7.62" width="0.1524" layer="91"/>
 <label x="96.52" y="7.62" size="1.778" layer="95"/>
+<pinref part="SW3" gate="G$1" pin="P$1"/>
+<wire x1="114.3" y1="7.62" x2="96.52" y2="7.62" width="0.1524" layer="91"/>
+</segment>
+</net>
+<net name="PB0" class="0">
+<segment>
+<pinref part="SW2" gate="G$1" pin="2"/>
+<wire x1="115.57" y1="-2.54" x2="96.52" y2="-2.54" width="0.1524" layer="91"/>
+<label x="96.52" y="-2.54" size="1.778" layer="95"/>
+</segment>
+<segment>
+<pinref part="U$1" gate="G$1" pin="PB0(SS)"/>
+<wire x1="76.2" y1="40.64" x2="91.44" y2="40.64" width="0.1524" layer="91"/>
+<label x="86.36" y="40.64" size="1.778" layer="95"/>
 </segment>
 </net>
@@
 will not be understood (or retained) with this version.
 </note>
+<note version="8.3" severity="warning">
+Since Version 8.3, EAGLE supports the association of 3D packages
+with devices in libraries, schematics, and board files. Those 3D
+packages will not be understood (or retained) with this version.
+</note>
 </compatibility>

Commit message: POIstick Rev 3
Parts:
- removed SW3: (no value), adafruit:SWITCH_PUSHBUTTONSOFTTOUCHSMD_SJ
- added LED13: APT2012SECK, microbuilder:LED0805
- added R15: 47, microbuilder:RESISTOR0805
- added S1: MOMENTARY-SWITCH-SPST-SMD-12MM, SparkFun-Switches:MOMENTARY-SWITCH-SPST-SMD-12MM
- added S3: (no value), SparkFun-Switches:SWITCH-SPDT-SMD-RIGHT-ANGLE
Connections:
- new net N$32: LED13.C, R15.1
- new net N$33: S3.O, U1.V+
- new net PD5: LED13.A, U$1.PD5(XCK/CTS)
- net GND: now also R15.2, S1.2; no longer SW3.P$2
- net PE6: now also S1.1; no longer SW3.P$1
- net VCC: now also S3.P; no longer U1.V+
Changed lines of the file:
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@@
 <part name="P+4" library="supply1" library_urn="urn:adsk.eagle:library:371" deviceset="VCC" device=""/>
 <part name="SW1" library="Wurth_Elektronik_Electromechanic_Switchs_rev15b" deviceset="431151015826" device=""/>
-<part name="SW3" library="adafruit" library_urn="urn:adsk.eagle:library:420" deviceset="SWITCH_PUSHBUTTON" device="SOFTTOUCHSMD_SJ"/>
 <part name="SW2" library="Wurth_Elektronik_Electromechanic_Switchs_rev15b" deviceset="431151015826" device=""/>
 <part name="C7" library="microbuilder" deviceset="CAP_CERAMIC" device="0805" value="0.1uF"/>
 <part name="GND9" library="supply1" library_urn="urn:adsk.eagle:library:371" deviceset="GND" device=""/>
 <part name="AREF" library="testpad" library_urn="urn:adsk.eagle:library:385" deviceset="PTR1" device="B1,27" package3d_urn="urn:adsk.eagle:package:27944/1" value="PTR1B1,27"/>
+<part name="S1" library="SparkFun-Switches" library_urn="urn:adsk.eagle:library:535" deviceset="MOMENTARY-SWITCH-SPST" device="-SMD-12MM" package3d_urn="urn:adsk.eagle:package:40166/1"/>
+<part name="LED13" library="microbuilder" deviceset="LED" device="0805" value="APT2012SECK"/>
+<part name="R15" library="microbuilder" deviceset="RESISTOR" device="0805" value="47"/>
+<part name="S3" library="SparkFun-Switches" library_urn="urn:adsk.eagle:library:535" deviceset="SWITCH-SPDT" device="-SMD-RIGHT-ANGLE" package3d_urn="urn:adsk.eagle:package:40179/1"/>
 </parts>
 <sheets>
@@
 <instance part="GND6" gate="1" x="60.96" y="106.68"/>
 <instance part="LED1" gate="G$1" x="142.24" y="106.68"/>
-<instance part="GND7" gate="1" x="182.88" y="43.18"/>
+<instance part="GND7" gate="1" x="182.88" y="25.4"/>
 <instance part="R3" gate="G$1" x="152.4" y="106.68"/>
 <instance part="LED2" gate="G$1" x="162.56" y="101.6"/>
@@
 <instance part="C2" gate="G$1" x="7.62" y="35.56" rot="R90"/>
 <instance part="GND8" gate="1" x="-35.56" y="7.62"/>
-<instance part="P+4" gate="VCC" x="-35.56" y="35.56"/>
+<instance part="P+4" gate="VCC" x="-35.56" y="48.26"/>
 <instance part="SW1" gate="G$1" x="119.38" y="25.4"/>
-<instance part="SW3" gate="G$1" x="119.38" y="7.62"/>
 <instance part="SW2" gate="G$1" x="119.38" y="-7.62" rot="MR0"/>
 <instance part="C7" gate="G$1" x="-7.62" y="15.24"/>
 <instance part="GND9" gate="1" x="-7.62" y="10.16"/>
 <instance part="AREF" gate="G$1" x="-12.7" y="20.32"/>
+<instance part="S1" gate="G$1" x="119.38" y="7.62"/>
+<instance part="LED13" gate="G$1" x="162.56" y="35.56"/>
+<instance part="R15" gate="G$1" x="172.72" y="35.56"/>
+<instance part="S3" gate="1" x="-35.56" y="43.18" rot="R270"/>
 </instances>
 <busses>
@@
 <segment>
 <pinref part="GND7" gate="1" pin="GND"/>
-<wire x1="182.88" y1="45.72" x2="182.88" y2="50.8" width="0.1524" layer="91"/>
+<wire x1="182.88" y1="27.94" x2="182.88" y2="35.56" width="0.1524" layer="91"/>
 <pinref part="R3" gate="G$1" pin="2"/>
+<wire x1="182.88" y1="35.56" x2="182.88" y2="50.8" width="0.1524" layer="91"/>
 <wire x1="182.88" y1="50.8" x2="182.88" y2="55.88" width="0.1524" layer="91"/>
 <wire x1="182.88" y1="55.88" x2="182.88" y2="60.96" width="0.1524" layer="91"/>
@@
 <wire x1="182.88" y1="50.8" x2="177.8" y2="50.8" width="0.1524" layer="91"/>
 <junction x="182.88" y="50.8"/>
+<pinref part="R15" gate="G$1" pin="2"/>
+<wire x1="177.8" y1="35.56" x2="182.88" y2="35.56" width="0.1524" layer="91"/>
+<junction x="182.88" y="35.56"/>
 </segment>
 <segment>
@@
 <segment>
 <label x="132.08" y="7.62" size="1.778" layer="95"/>
-<pinref part="SW3" gate="G$1" pin="P$2"/>
 <wire x1="124.46" y1="7.62" x2="137.16" y2="7.62" width="0.1524" layer="91"/>
+<pinref part="S1" gate="G$1" pin="2"/>
 </segment>
 <segment>
@@
 </segment>
 <segment>
-<pinref part="U1" gate="CR2032" pin="V+"/>
 <pinref part="P+4" gate="VCC" pin="VCC"/>
-<wire x1="-35.56" y1="33.02" x2="-35.56" y2="27.94" width="0.1524" layer="91"/>
+<pinref part="S3" gate="1" pin="P"/>
 </segment>
 </net>
@@
 <segment>
 <label x="96.52" y="7.62" size="1.778" layer="95"/>
-<pinref part="SW3" gate="G$1" pin="P$1"/>
 <wire x1="114.3" y1="7.62" x2="96.52" y2="7.62" width="0.1524" layer="91"/>
+<pinref part="S1" gate="G$1" pin="1"/>
 </segment>
 </net>
@@
 </segment>
 </net>
+<net name="PD5" class="0">
+<segment>
+<pinref part="U$1" gate="G$1" pin="PD5(XCK/CTS)"/>
+<wire x1="76.2" y1="30.48" x2="91.44" y2="30.48" width="0.1524" layer="91"/>
+<label x="86.36" y="30.48" size="1.778" layer="95"/>
+</segment>
+<segment>
+<pinref part="LED13" gate="G$1" pin="A"/>
+<wire x1="157.48" y1="35.56" x2="142.24" y2="35.56" width="0.1524" layer="91"/>
+<label x="142.24" y="35.56" size="1.778" layer="95"/>
+</segment>
+</net>
+<net name="N$32" class="0">
+<segment>
+<pinref part="LED13" gate="G$1" pin="C"/>
+<pinref part="R15" gate="G$1" pin="1"/>
+<wire x1="167.64" y1="35.56" x2="165.1" y2="35.56" width="0.1524" layer="91"/>
+</segment>
+</net>
+<net name="N$33" class="0">
+<segment>
+<pinref part="U1" gate="CR2032" pin="V+"/>
+<pinref part="S3" gate="1" pin="O"/>
+<wire x1="-35.56" y1="27.94" x2="-35.56" y2="35.56" width="0.1524" layer="91"/>
+<wire x1="-35.56" y1="35.56" x2="-33.02" y2="38.1" width="0.1524" layer="91"/>
+</segment>
+</net>

Commit message: POIstick Rev 7
Parts:
- PTCFUSE: value 250mA -> 500mA
- renumbered F2 to PTCFUSE
Changed lines of the file:
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@@
 <part name="R2" library="microbuilder" deviceset="RESISTOR" device="0805" value="22"/>
 <part name="GND1" library="supply1" library_urn="urn:adsk.eagle:library:371" deviceset="GND" device=""/>
-<part name="F2" library="microbuilder" deviceset="PTC" device="1206" value="250mA"/>
+<part name="PTCFUSE" library="microbuilder" deviceset="PTC" device="1206" value="500mA"/>
 <part name="SUPPLY1" library="supply2" library_urn="urn:adsk.eagle:library:372" deviceset="+5V" device=""/>
 <part name="SUPPLY2" library="supply2" library_urn="urn:adsk.eagle:library:372" deviceset="+5V" device=""/>
@@
 <instance part="R2" gate="G$1" x="-10.16" y="60.96"/>
 <instance part="GND1" gate="1" x="-25.4" y="53.34"/>
-<instance part="F2" gate="G$1" x="-25.4" y="78.74" rot="R270"/>
+<instance part="PTCFUSE" gate="G$1" x="-25.4" y="78.74" rot="R270"/>
 <instance part="SUPPLY1" gate="+5V" x="-25.4" y="86.36"/>
 <instance part="SUPPLY2" gate="+5V" x="12.7" y="91.44"/>
@@
 <pinref part="CN1" gate="G$1" pin="VBUS"/>
 <wire x1="-27.94" y1="66.04" x2="-25.4" y2="66.04" width="0.1524" layer="91"/>
-<pinref part="F2" gate="G$1" pin="1"/>
+<pinref part="PTCFUSE" gate="G$1" pin="1"/>
 <wire x1="-25.4" y1="66.04" x2="-25.4" y2="73.66" width="0.1524" layer="91"/>
 </segment>
@@
 <net name="+5V" class="0">
 <segment>
-<pinref part="F2" gate="G$1" pin="2"/>
+<pinref part="PTCFUSE" gate="G$1" pin="2"/>
 <pinref part="SUPPLY1" gate="+5V" pin="+5V"/>
 </segment>
@@
 <pinref part="LED7" gate="G$1" pin="A"/>
 <pinref part="U$1" gate="G$1" pin="PE2(!HWB)"/>
-<wire x1="137.16" y1="76.2" x2="76.2" y2="73.66" width="0.1524" layer="91"/>
+<wire x1="137.16" y1="76.2" x2="106.68" y2="76.2" width="0.1524" layer="91"/>
+<wire x1="106.68" y1="76.2" x2="106.68" y2="73.66" width="0.1524" layer="91"/>
+<wire x1="106.68" y1="73.66" x2="76.2" y2="73.66" width="0.1524" layer="91"/>
 </segment>
 </net>
@@
 <segment>
 <pinref part="LED8" gate="G$1" pin="A"/>
-<wire x1="157.48" y1="71.12" x2="137.16" y2="71.12" width="0.1524" layer="91"/>
 <pinref part="U$1" gate="G$1" pin="PC7(ICP3/CLK0/OC4A)"/>
-<wire x1="76.2" y1="63.5" x2="137.16" y2="71.12" width="0.1524" layer="91"/>
+<wire x1="76.2" y1="63.5" x2="109.22" y2="63.5" width="0.1524" layer="91"/>
+<wire x1="109.22" y1="63.5" x2="109.22" y2="71.12" width="0.1524" layer="91"/>
+<wire x1="109.22" y1="71.12" x2="157.48" y2="71.12" width="0.1524" layer="91"/>
 </segment>
 </net>
@@
 <segment>
 <pinref part="LED10" gate="G$1" pin="A"/>
-<wire x1="157.48" y1="60.96" x2="137.16" y2="60.96" width="0.1524" layer="91"/>
 <pinref part="U$1" gate="G$1" pin="PB6(OC1B/OC4B/ADC13)"/>
-<wire x1="137.16" y1="60.96" x2="76.2" y2="55.88" width="0.1524" layer="91"/>
+<wire x1="157.48" y1="60.96" x2="106.68" y2="60.96" width="0.1524" layer="91"/>
+<wire x1="106.68" y1="60.96" x2="106.68" y2="55.88" width="0.1524" layer="91"/>
+<wire x1="106.68" y1="55.88" x2="76.2" y2="55.88" width="0.1524" layer="91"/>
 </segment>
 </net>
@@
 <pinref part="LED11" gate="G$1" pin="A"/>
 <pinref part="U$1" gate="G$1" pin="PB5(OC1A/ADC12/!OC4B)"/>
-<wire x1="137.16" y1="55.88" x2="76.2" y2="53.34" width="0.1524" layer="91"/>
+<wire x1="137.16" y1="55.88" x2="109.22" y2="55.88" width="0.1524" layer="91"/>
+<wire x1="109.22" y1="55.88" x2="109.22" y2="53.34" width="0.1524" layer="91"/>
+<wire x1="109.22" y1="53.34" x2="76.2" y2="53.34" width="0.1524" layer="91"/>
 </segment>
 </net>
@@
 <segment>
 <pinref part="U$1" gate="G$1" pin="PE6(INT.6/AIN0)"/>
-<wire x1="76.2" y1="71.12" x2="86.36" y2="71.12" width="0.1524" layer="91"/>
-<label x="81.28" y="71.12" size="1.778" layer="95"/>
+<wire x1="76.2" y1="71.12" x2="91.44" y2="71.12" width="0.1524" layer="91"/>
+<label x="86.36" y="71.12" size="1.778" layer="95"/>
 </segment>
 <segment>
@@
 <segment>
 <pinref part="LED13" gate="G$1" pin="A"/>
-<wire x1="157.48" y1="35.56" x2="142.24" y2="35.56" width="0.1524" layer="91"/>
-<label x="142.24" y="35.56" size="1.778" layer="95"/>
-</segment>
-</net>
+<wire x1="157.48" y1="35.56" x2="147.32" y2="35.56" width="0.1524" layer="91"/>
+<label x="147.32" y="35.56" size="1.778" layer="95"/>
+</segment>
+</net>

Commit message: UCAP 0.1uF, replace 3.3V -> VCC
Parts:
- C8: value 0.1uF -> 1uF
Connections:
- net +3V3 renamed N$34
Changed lines of the file:
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@@
 <part name="GND3" library="supply1" library_urn="urn:adsk.eagle:library:371" deviceset="GND" device=""/>
 <part name="X1" library="adafruit" deviceset="XTAL" device="NX5032" value="2MHz"/>
-<part name="+3V1" library="supply1" library_urn="urn:adsk.eagle:library:371" deviceset="+3V3" device=""/>
 <part name="GND4" library="supply1" library_urn="urn:adsk.eagle:library:371" deviceset="GND" device=""/>
 <part name="GND5" library="supply1" library_urn="urn:adsk.eagle:library:371" deviceset="GND" device=""/>
@@
 <part name="R14" library="microbuilder" deviceset="RESISTOR" device="0805" value="47"/>
 <part name="U1" library="CR2032-SnapDragon" deviceset="CR2032-SNAPDRAGON" device="CR2032"/>
-<part name="C8" library="microbuilder" deviceset="CAP_CERAMIC" device="0805" value="0.1uF"/>
+<part name="C8" library="microbuilder" deviceset="CAP_CERAMIC" device="0805" value="1uF"/>
 <part name="C3" library="microbuilder" deviceset="CAP_CERAMIC" device="0805" value="0.1uF"/>
 <part name="C4" library="microbuilder" deviceset="CAP_CERAMIC" device="0805" value="0.1uF"/>
@@
 <instance part="GND3" gate="1" x="-2.54" y="40.64" rot="R270"/>
 <instance part="X1" gate="G$1" x="17.78" y="40.64" rot="R90"/>
-<instance part="+3V1" gate="G$1" x="-5.08" y="58.42"/>
 <instance part="GND4" gate="1" x="-5.08" y="45.72"/>
 <instance part="GND5" gate="1" x="-33.02" y="106.68"/>
@@
 </segment>
 </net>
-<net name="+3V3" class="0">
-<segment>
-<pinref part="U$1" gate="G$1" pin="UCAP"/>
-<pinref part="+3V1" gate="G$1" pin="+3V3"/>
-<wire x1="27.94" y1="55.88" x2="-5.08" y2="55.88" width="0.1524" layer="91"/>
-<junction x="-5.08" y="55.88"/>
-<pinref part="C8" gate="G$1" pin="P$1"/>
-</segment>
-</net>
 <net name="AREF" class="0">
 <segment>
@@
 </segment>
 </net>
+<net name="N$34" class="0">
+<segment>
+<pinref part="U$1" gate="G$1" pin="UCAP"/>
+<wire x1="27.94" y1="55.88" x2="-5.08" y2="55.88" width="0.1524" layer="91"/>
+<pinref part="C8" gate="G$1" pin="P$1"/>
+</segment>
+</net>
