File: POIstick/POIstick2.brd (EAGLE design)
At the start: 87.3 x 22.9 mm, 39 parts, among them U1 CR2032-SNAPDRAGONCR2032, X1 8MHz

Commit message: initial V2
Parts:
- removed F2: (no value), adafruit:R1206
- added AREF: PTR1B1,27, testpad:B1,27
- added C8: 1uF, microbuilder:0805
- added LED13: APT2012SECK, microbuilder:CHIPLED_0805
- added PTCFUSE: 500mA, microbuilder:1206
- added R15: 47, microbuilder:0805
- added S1: MOMENTARY-SWITCH-SPST-SMD-12MM, SparkFun-Switches:TACTILE_SWITCH_SMD_12MM
- added S3: (no value), SparkFun-Switches:SWITCH_SPST_SMD_A
- added SW1, SW2: 431151015826, Wurth_Elektronik_Electromechanic_Switchs_rev15b:431181015816
- C1, C2, C4, C5: device rcl:C1206 -> microbuilder:0805
- C3: value (none) -> 0.1uF; device rcl:C1206 -> microbuilder:0805
- C6: value 0.1uF -> 10uF; device rcl:C1206 -> microbuilder:EIA3216-18/A-W
- C7: value 10uF -> 0.1uF; device resistor:CT3216 -> microbuilder:0805
- LED1: value (none) -> Orange APT2012SECK; device adafruit:CHIPLED_0805 -> microbuilder:CHIPLED_0805
- LED10, LED11, LED12, LED2, LED3, LED4, LED5, LED6, LED7, LED8, LED9: value (none) -> APT2012SECK; device adafruit:CHIPLED_0805 -> microbuilder:CHIPLED_0805
- R1, R2: device adafruit:R0805 -> microbuilder:0805
- R10, R11, R12, R13, R14, R3, R4, R5, R6, R7, R8, R9: value 22 -> 47; device adafruit:R0805 -> microbuilder:0805
- X1: value 8MHz -> 2MHz
- moved C7 18.7 mm to (44.5, 63.5), turned to 180 degrees
- moved C5 10.2 mm to (73.7, 59.7), turned to 0 degrees
- moved C1 7.65 mm to (88.9, 73.0), turned to 180 degrees
- moved C4 6.84 mm to (64.8, 61.0)
- moved C2 4.77 mm to (88.9, 64.1), turned to 180 degrees
- moved C3 2.84 mm to (68.6, 62.2), turned to 0 degrees
- moved X1 2.84 mm to (88.9, 68.6)
- moved C6 1.80 mm to (63.5, 69.8), turned to 0 degrees
- moved U1 1.40 mm to (30.6, 68.6)
- moved R3 0.68 mm to (42.8, 73.0)
- moved R4 0.65 mm to (47.6, 73.0)
- moved R10 0.63 mm to (78.0, 73.0)
- moved R11 0.63 mm to (83.1, 73.0)
- moved R12 0.63 mm to (88.1, 73.0)
- moved R13 0.63 mm to (93.2, 73.0)
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Connections:
- removed net +3V3: C3.2, U$1.6
- new net N$32: LED13.C, R15.1
- new net N$33: S3.1, U1.V+
- new net N$34: C8.1, U$1.6
- new net PB0: SW2.2, U$1.8
- new net PD5: LED13.A, U$1.22
- new net PE6: S1.1, U$1.1
- net +5V: now also C5.1, C6.+, PTCFUSE.2; no longer C6.2, C7.-, F2.2
- net AREF: now also AREF.TP, C7.1
- net GND: now also C3.2, C4.2, C5.2, C6.-, C7.2, C8.2, R15.2, S1.3, SW1.2, SW2.1, U1.V-; no longer C3.1, C4.1, C5.1, C6.1, C7.+
- net N$5: now also PTCFUSE.1; no longer F2.1
- net RST: now also SW1.1
- net VCC: now also C3.1, C4.1, S3.2; no longer C4.2, C5.2
Routing:
- net GND: track 77.2 -> 168.4 mm, vias 4 -> 9
- net VCC: track 29.8 -> 111.2 mm, vias 0 -> 3
- net RST: track 0.00 -> 60.4 mm, vias 0 -> 1
- net PE6: track 0.00 -> 53.4 mm
- net PB0: track 0.00 -> 38.7 mm, vias 0 -> 2
- net AREF: track 0.00 -> 31.4 mm, vias 0 -> 2
- net N$33: track 0.00 -> 31.3 mm
- net MOSI: track 0.00 -> 24.0 mm, vias 0 -> 1
- net MISO: track 0.00 -> 22.4 mm, vias 0 -> 1
- net +5V: track 7.43 -> 29.8 mm, vias 0 -> 2
- net SCK: track 0.00 -> 21.5 mm, vias 0 -> 1
- net N$7: track 0.00 -> 14.5 mm
- net N$2: track 0.00 -> 13.1 mm
- net N$1: track 0.00 -> 12.9 mm
- net N$34: track 0.00 -> 11.0 mm, vias 0 -> 2
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- added copper zone on layer 1, net GND
- added copper zone on layer 16, net GND
Other:
- board size 87.3 x 22.9 mm -> 86 x 22.9 mm
- board text added: "...running!"
- board text added: "ATmega32U4"
- board text added: "CONF"
- board text added: "GND"
- board text added: "MISO"
- board text added: "MOSI"
- board text added: "POIstick"
- board text added: "RST"
- board text added: "SCK"
- board text added: "START!"
- board text added: "VCC"
- board text added: "Version 1.0 (C) AE@2017"

Commit message: WIP
Parts:
- removed LED1: Orange APT2012SECK, microbuilder:CHIPLED_0805
- removed LED10, LED11, LED12, LED2, LED3, LED4, LED5, LED6, LED7, LED8, LED9: APT2012SECK, microbuilder:CHIPLED_0805
- removed R10, R11, R12, R13, R14, R3, R4, R5, R6, R7, R8, R9: 47, microbuilder:0805
- added C10, C11, C12, C13, C14, C15, C16, C17, C18, C9: 0.1uF, microbuilder:0805
- added D1, D10, D2, D3, D4, D5, D6, D7, D8, D9: WS2812B, SparkFun-LED:WS2812B
- moved C1 39.6 mm to (85.1, 33.7)
- moved C2 39.6 mm to (85.1, 24.8)
- moved C4 39.6 mm to (61.0, 21.6)
- moved C7 39.6 mm to (40.6, 24.1)
- moved CN1 39.6 mm to (52.5, 22.4)
- moved PTCFUSE 39.6 mm to (52.2, 31.8)
- moved R2 39.6 mm to (63.5, 27.9)
- moved S3 39.6 mm to (42.5, 19.7)
- moved SW1 39.6 mm to (33.7, 36.8)
- moved SW2 39.6 mm to (33.7, 21.6)
- moved AREF 39.6 mm to (44.7, 27.3)
- moved C3 39.6 mm to (64.8, 22.9)
- moved C5 39.6 mm to (69.8, 20.3)
- moved C8 39.6 mm to (64.8, 20.3)
- moved ISP 39.6 mm to (91.2, 21.3)
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Connections:
- removed net N$20: LED7.C, R9.1
- removed net N$21: LED7.A, U$1.33
- removed net N$22: LED8.C, R10.1
- removed net N$23: LED8.A, U$1.32
- removed net N$24: LED9.C, R11.1
- removed net N$25: LED9.A, U$1.31
- removed net N$26: LED10.C, R12.1
- removed net N$27: LED10.A, U$1.30
- removed net N$28: LED11.C, R13.1
- removed net N$29: LED11.A, U$1.29
- removed net N$30: LED12.C, R14.1
- removed net N$31: LED12.A, U$1.28
- net GND: now also C10.2, C11.2, C12.2, C13.2, C14.2, C15.2, C16.2, C17.2, C18.2, C9.2, D1.3, D10.3, D2.3, D3.3, D4.3, D5.3, D6.3, D7.3, D8.3, D9.3; no longer R10.2, R11.2, R12.2, R13.2, R14.2, R3.2, R4.2, R5.2, R6.2, R7.2, R8.2, R9.2
- net N$10: now also D3.2, D4.4; no longer LED2.C, R4.1
- net N$11: now also D4.2, D5.4; no longer LED1.A, U$1.36
- net N$12: now also D5.2, D6.4; no longer LED3.C, R5.1
- net N$13: now also D6.2, D7.4; no longer LED3.A, U$1.38
- net N$14: now also D7.2, D8.4; no longer LED4.C, R6.1
- net N$15: now also D8.2, D9.4; no longer LED4.A, U$1.39
- net N$16: now also D10.4, D9.2; no longer LED5.C, R7.1
- net N$17: now also D1.4; no longer LED5.A, U$1.40
- net N$18: now also R1.2; no longer LED6.C, R8.1
- net N$19: now also R2.2; no longer LED6.A, U$1.41
- net N$3: now also U$1.3; no longer R1.2, U$1.4
- net N$4: now also U$1.4; no longer R2.2, U$1.3
- net N$8: now also D1.2, D2.4; no longer LED1.C, R3.1
- net N$9: now also D2.2, D3.4; no longer LED2.A, U$1.37
- net VCC: now also C10.1, C11.1, C12.1, C13.1, C14.1, C15.1, C16.1, C17.1, C18.1, C9.1, D1.1, D10.1, D2.1, D3.1, D4.1, D5.1, D6.1, D7.1, D8.1, D9.1
Routing:
- net GND: track 168.4 -> 98.9 mm, vias 9 -> 1
- net N$11: track 35.3 -> 0.00 mm, vias 1 -> 0
- net N$9: track 29.1 -> 0.00 mm, vias 1 -> 0
- net N$13: track 23.4 -> 0.00 mm, vias 1 -> 0
- net N$31: track 19.2 -> 0.00 mm, vias 1 -> 0
- net N$15: track 18.0 -> 0.00 mm, vias 1 -> 0
- net N$29: track 14.5 -> 0.00 mm, vias 1 -> 0
- net N$17: track 13.2 -> 0.00 mm, vias 1 -> 0
- net AREF: track 31.4 -> 19.4 mm, vias 2 -> 0
- net VCC: track 111.2 -> 101.0 mm, vias 3 -> 1
- net N$27: track 9.69 -> 0.00 mm, vias 1 -> 0
- net N$19: track 8.80 -> 0.00 mm, vias 1 -> 0
- net N$21: track 7.16 -> 0.00 mm, vias 1 -> 0
- net +5V: track 29.8 -> 23.6 mm, vias 2 -> 0
- net N$25: track 6.16 -> 0.00 mm, vias 1 -> 0
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- removed copper zone on layer 1, net GND
- removed copper zone on layer 16, net GND
Other:
- board size 86 x 22.9 mm -> 98.7 x 22.9 mm

Commit message: WIP
Parts:
- added C19: 4.7uF, microbuilder:0805
- added C20: 10uF, microbuilder:0805
- added L1: 4.7uH, WE-TPC:WE-TPC_3816
- added R3: 976K, microbuilder:0805
- added R4: 309K, microbuilder:0805
- added U$2: MCP1623/24, MCP1623:SOT95P300X120-6N
- X1: value 2MHz -> 8MHz
- moved C3 11.4 mm to (76.2, 22.9)
- moved C5 11.4 mm to (81.3, 20.3)
- moved C6 11.4 mm to (71.1, 30.5)
- moved C8 11.4 mm to (76.2, 20.3)
- moved R1 11.4 mm to (74.9, 25.4)
- moved R2 11.4 mm to (74.9, 27.9)
- moved U$1 11.4 mm to (85.1, 29.2)
- moved AREF 11.4 mm to (56.1, 27.3)
- moved C4 11.4 mm to (72.4, 21.6)
- moved C7 11.4 mm to (52.1, 24.1)
- moved CN1 11.4 mm to (63.9, 22.4)
- moved PTCFUSE 11.4 mm to (63.6, 31.8)
- moved C1 11.4 mm to (96.5, 33.7)
- moved C2 11.4 mm to (96.5, 24.8)
- moved ISP 11.4 mm to (102.6, 21.3)
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Connections:
- removed net N$18: R1.2
- removed net N$4: U$1.4
- new net USB_D+: R1.2, U$1.4
- new net USB_D-: R2.2, U$1.3
- new net VIN: C19.1, L1.1, S3.2, U$2.3, U$2.6
- net GND: now also C19.2, C20.2, R4.2, U$2.2
- net N$19: now also L1.2, U$2.1; no longer R2.2
- net N$3: now also R3.2, R4.1, U$2.4; no longer U$1.3
- net VCC: now also C20.1, R3.1, U$2.5; no longer S3.2
Routing:
- net VCC: track 101.0 -> 240.9 mm, vias 1 -> 0
- net PB0: track 38.7 -> 87.9 mm
- net GND: track 98.9 -> 140.8 mm, vias 1 -> 0
- net RST: track 60.4 -> 92.9 mm
- net MOSI: track 24.0 -> 46.8 mm
- net SCK: track 21.5 -> 41.9 mm
- net MISO: track 22.4 -> 40.5 mm
- net PD5: track 10.8 -> 27.8 mm
- net VIN: track 0.00 -> 15.2 mm
- net N$34: track 11.0 -> 21.8 mm
- net PE6: track 53.4 -> 63.2 mm
- net N$19: track 0.00 -> 7.68 mm
- net N$3: track 0.00 -> 6.48 mm
- net N$15: track 0.00 -> 6.46 mm
- net N$13: track 0.00 -> 6.46 mm
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
Commit message: WIP
Parts:
- added D11, D12: (no value), eagle-ltspice:DIODE_SMB
- added Q2: (no value), transistor-power:SO-08
- added R5: 10k, microbuilder:0805
Connections:
- new net N$20: D12.A, Q2.5, Q2.6, Q2.7, Q2.8
- new net N$4: C20.1, Q2.1, Q2.2, Q2.3, R3.1, U$2.5
- net +5V: now also D11.A, Q2.4, R5.1
- net GND: now also R5.2
- net VCC: now also D11.C, D12.C; no longer C20.1, R3.1, U$2.5
Routing:
- net VCC: track 240.9 -> 230.0 mm
- net N$4: track 0.00 -> 7.57 mm
Changed lines of the file:
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@@
 </element>
 <element name="C20" library="microbuilder" package="0805" value="10uF" x="56.642" y="25.527" rot="MR90"/>
+<element name="Q2" library="transistor-power" library_urn="urn:adsk.eagle:library:400" package="SO-08" package3d_urn="urn:adsk.eagle:package:29505/2" value="" x="2.54" y="10.16"/>
+<element name="D11" library="eagle-ltspice" library_urn="urn:adsk.eagle:library:217" package="DIODE_SMB" package3d_urn="urn:adsk.eagle:package:13312/1" value="" x="5.08" y="-1.27">
+<attribute name="SPICEMODEL" value="NONE" x="5.08" y="-1.27" size="1.778" layer="27" display="off"/>
+<attribute name="SPICEPREFIX" value="D" x="5.08" y="-1.27" size="1.778" layer="27" display="off"/>
+<attribute name="SPICETYPE" value="diode" x="5.08" y="-1.27" size="1.778" layer="27" display="off"/>
+</element>
+<element name="R5" library="microbuilder" package="0805" value="10k" x="1.27" y="-6.35"/>
+<element name="D12" library="eagle-ltspice" library_urn="urn:adsk.eagle:library:217" package="DIODE_SMB" package3d_urn="urn:adsk.eagle:package:13312/1" value="" x="5.08" y="-13.97">
+<attribute name="SPICEMODEL" value="NONE" x="5.08" y="-13.97" size="1.778" layer="27" display="off"/>
+<attribute name="SPICEPREFIX" value="D" x="5.08" y="-13.97" size="1.778" layer="27" display="off"/>
+<attribute name="SPICETYPE" value="diode" x="5.08" y="-13.97" size="1.778" layer="27" display="off"/>
+</element>
 </elements>
 <signals>
@@
 <wire x1="53.34" y1="27.94" x2="54.61" y2="27.94" width="0.3048" layer="16"/>
 <wire x1="54.61" y1="27.94" x2="56.642" y2="26.477" width="0.3048" layer="16"/>
+<contactref element="R5" pad="2"/>
 <wire x1="100.654584375" y1="34.487584375" x2="104.47" y2="32.983" width="0" layer="19" extent="1-16"/>
 <wire x1="99.06" y1="34.29" x2="100.654584375" y2="34.487584375" width="0" layer="19" extent="1-1"/>
@@
 <wire x1="66.548" y1="27.4094" x2="66.37" y2="30.495" width="0" layer="19" extent="1-16"/>
 <wire x1="60.02" y1="30.495" x2="66.355" y2="30.48" width="0" layer="19" extent="16-16"/>
-<wire x1="56.642" y1="26.477" x2="60.02" y2="30.495" width="0" layer="19" extent="16-16"/>
+<wire x1="56.642" y1="26.477" x2="60.005" y2="30.48" width="0" layer="19" extent="16-16"/>
 <wire x1="50.8" y1="27.94" x2="50.378265625" y2="26.5007625" width="0" layer="19" extent="1-16"/>
 <wire x1="49.85" y1="21.59" x2="50.43" y2="23.44" width="0" layer="19" extent="1-16"/>
@@
 <wire x1="39.445303125" y1="36.5125" x2="47.32" y2="32.983" width="0" layer="19" extent="16-16"/>
 <wire x1="35.955" y1="34.98" x2="39.445303125" y2="36.5125" width="0" layer="19" extent="1-16"/>
+<wire x1="2.22" y1="-6.35" x2="25.868" y2="22.362" width="0" layer="19" extent="1-1"/>
 </signal>
 <signal name="N$1">
@@
 <wire x1="80.33" y1="23.318628125" x2="81.554465625" y2="24.54309375" width="0.254" layer="1"/>
 <wire x1="72.595" y1="30.48" x2="74.93" y2="30.099" width="0.254" layer="1"/>
+<contactref element="Q2" pad="4"/>
+<contactref element="R5" pad="1"/>
+<contactref element="D11" pad="A"/>
 <wire x1="74.93" y1="30.099" x2="78.7260375" y2="27.371521875" width="0" layer="19" extent="1-1"/>
+<wire x1="4.445" y1="7.56" x2="65.027" y2="31.75" width="0" layer="19" extent="1-1"/>
+<wire x1="7.28" y1="-1.27" x2="4.445" y2="7.56" width="0" layer="19" extent="1-1"/>
+<wire x1="0.32" y1="-6.35" x2="7.28" y2="-1.27" width="0" layer="19" extent="1-1"/>
 </signal>
 <signal name="VCC">
@@
 <wire x1="88.57" y1="38.137" x2="87.63" y2="39.37" width="0.3048" layer="16"/>
 <wire x1="94.92" y1="38.137" x2="93.98" y2="39.37" width="0.3048" layer="16"/>
-<contactref element="R3" pad="1"/>
-<contactref element="U$2" pad="5"/>
-<contactref element="C20" pad="1"/>
-<wire x1="53.748" y1="24.92035" x2="53.89585" y2="25.0682" width="0.3048" layer="16"/>
-<wire x1="53.89585" y1="25.0682" x2="54.66375" y2="25.0682" width="0.3048" layer="16"/>
-<wire x1="54.66375" y1="25.0682" x2="54.8116" y2="24.92035" width="0.3048" layer="16"/>
-<wire x1="54.8116" y1="24.92035" x2="54.8116" y2="24.284778125" width="0.3048" layer="16"/>
-<wire x1="54.8116" y1="24.284778125" x2="56.642" y2="24.577" width="0.3048" layer="16"/>
-<wire x1="53.34" y1="24.1808" x2="53.748" y2="24.598578125" width="0.3048" layer="16"/>
-<wire x1="53.748" y1="24.598578125" x2="53.748" y2="24.92035" width="0.3048" layer="16"/>
-<wire x1="56.642" y1="24.577" x2="56.83" y2="21.59" width="0.3048" layer="16"/>
-<wire x1="56.83" y1="21.59" x2="56.83" y2="24.90805" width="0.3048" layer="16"/>
 <wire x1="56.83" y1="24.90805" x2="57.6444" y2="25.72245" width="0.3048" layer="16"/>
 <wire x1="57.6444" y1="30.0194" x2="58.105" y2="30.48" width="0.3048" layer="16"/>
 <wire x1="57.6444" y1="25.72245" x2="57.6444" y2="30.0194" width="0.3048" layer="16"/>
+<contactref element="D11" pad="C"/>
+<contactref element="D12" pad="C"/>
 <wire x1="89.855" y1="30.48" x2="89.31114375" y2="30.57685625" width="0" layer="19" extent="1-16"/>
 <wire x1="73.787" y1="23.749" x2="70.805" y2="30.48" width="0" layer="19" extent="1-16"/>
+<wire x1="2.88" y1="-1.27" x2="45.405" y2="30.48" width="0" layer="19" extent="1-16"/>
+<wire x1="2.88" y1="-13.97" x2="2.88" y2="-1.27" width="0" layer="19" extent="1-1"/>
 </signal>
 <signal name="N$6">
@@
 <wire x1="50.7864" y1="26.65345625" x2="52.4002" y2="26.6192" width="0.3048" layer="16"/>
 </signal>
+<signal name="N$4">
+<contactref element="R3" pad="1"/>
+<contactref element="U$2" pad="5"/>
+<contactref element="C20" pad="1"/>
+<wire x1="53.748" y1="24.92035" x2="53.89585" y2="25.0682" width="0.3048" layer="16"/>
+<wire x1="53.89585" y1="25.0682" x2="54.66375" y2="25.0682" width="0.3048" layer="16"/>
+<wire x1="54.66375" y1="25.0682" x2="54.8116" y2="24.92035" width="0.3048" layer="16"/>
+<wire x1="54.8116" y1="24.92035" x2="54.8116" y2="24.284778125" width="0.3048" layer="16"/>
+<wire x1="54.8116" y1="24.284778125" x2="56.642" y2="24.577" width="0.3048" layer="16"/>
+<wire x1="53.34" y1="24.1808" x2="53.748" y2="24.598578125" width="0.3048" layer="16"/>
+<wire x1="53.748" y1="24.598578125" x2="53.748" y2="24.92035" width="0.3048" layer="16"/>
+<wire x1="56.642" y1="24.577" x2="56.83" y2="21.59" width="0.3048" layer="16"/>
+<contactref element="Q2" pad="1"/>
+<contactref element="Q2" pad="3"/>
+<contactref element="Q2" pad="2"/>
+<wire x1="3.175" y1="7.56" x2="53.34" y2="24.1808" width="0" layer="19" extent="1-16"/>
+<wire x1="1.905" y1="7.56" x2="3.175" y2="7.56" width="0" layer="19" extent="1-1"/>
+<wire x1="0.635" y1="7.56" x2="1.905" y2="7.56" width="0" layer="19" extent="1-1"/>
+</signal>
+<signal name="N$20">
+<contactref element="Q2" pad="6"/>
+<contactref element="Q2" pad="5"/>
+<contactref element="Q2" pad="8"/>
+<contactref element="Q2" pad="7"/>
+<contactref element="D12" pad="A"/>
+<wire x1="4.445" y1="12.76" x2="3.175" y2="12.76" width="0" layer="19" extent="1-1"/>
+<wire x1="1.905" y1="12.76" x2="3.175" y2="12.76" width="0" layer="19" extent="1-1"/>
+<wire x1="0.635" y1="12.76" x2="1.905" y2="12.76" width="0" layer="19" extent="1-1"/>
+<wire x1="7.28" y1="-13.97" x2="4.445" y2="12.76" width="0" layer="19" extent="1-1"/>
+</signal>
 </signals>
