File: POIstick/POIstick2.brd (EAGLE design)
At the start: 98.7 x 22.9 mm, 53 parts, among them SW1 431151015826, SW2 431151015826, U1 CR2032-SNAPDRAGONCR2032, X1 8MHz

Commit message: WIP
Parts:
- added C21: 0.1uF, rcl:C1206
- added C22: 10uF, rcl:C1206
- added R6, R7, R8: 10k, microbuilder:0805
- added U2: LIS3DH, SparkFun-Sensors:LGA-16-3X3
Connections:
- new net ACCEL_INT1: U$1.20, U2.11
- new net ACCEL_INT2: U$1.21, U2.9
- new net N$18: R8.2, U2.8
- new net N$23: R6.1, R7.1, U2.1
- new net SCL: R7.2, U$1.18, U2.6
- new net SDA: R6.2, U$1.19, U2.4
- new net V_USB: PTCFUSE.2, U$1.2, U$1.7
- net +5V: no longer PTCFUSE.2, U$1.2, U$1.7
- net GND: now also C21.2, C22.2, U2.10, U2.12, U2.13, U2.15, U2.16, U2.5, U2.7
- net VCC: now also C21.1, C22.1, R8.1, U2.14
Routing:
- net +5V: track 23.6 -> 12.3 mm
- net V_USB: track 0.00 -> 7.42 mm
Changed lines of the file:
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@@
 <attribute name="SPICETYPE" value="diode" x="5.08" y="-13.97" size="1.778" layer="27" display="off"/>
 </element>
+<element name="U2" library="SparkFun-Sensors" package="LGA-16-3X3" value="LIS3DH" x="-5.08" y="-12.7">
+<attribute name="PROD_ID" value="IC-13419" x="-5.08" y="-12.7" size="1.778" layer="27" display="off"/>
+<attribute name="SF_ID" value="N/A" x="-5.08" y="-12.7" size="1.778" layer="27" display="off"/>
+</element>
+<element name="C22" library="rcl" library_urn="urn:adsk.eagle:library:334" package="C1206" package3d_urn="urn:adsk.eagle:package:23618/2" value="10uF" x="-5.08" y="-25.4"/>
+<element name="C21" library="rcl" library_urn="urn:adsk.eagle:library:334" package="C1206" package3d_urn="urn:adsk.eagle:package:23618/2" value="0.1uF" x="-5.08" y="-31.75"/>
+<element name="R6" library="microbuilder" package="0805" value="10k" x="-5.08" y="-38.1"/>
+<element name="R7" library="microbuilder" package="0805" value="10k" x="-5.08" y="-43.18"/>
+<element name="R8" library="microbuilder" package="0805" value="10k" x="-5.08" y="-48.26"/>
 </elements>
 <signals>
@@
 <wire x1="54.61" y1="27.94" x2="56.642" y2="26.477" width="0.3048" layer="16"/>
 <contactref element="R5" pad="2"/>
+<contactref element="C21" pad="2"/>
+<contactref element="C22" pad="2"/>
+<contactref element="U2" pad="5"/>
+<contactref element="U2" pad="10"/>
+<contactref element="U2" pad="12"/>
+<contactref element="U2" pad="16"/>
+<contactref element="U2" pad="15"/>
+<contactref element="U2" pad="13"/>
+<contactref element="U2" pad="7"/>
 <wire x1="100.654584375" y1="34.487584375" x2="104.47" y2="32.983" width="0" layer="19" extent="1-16"/>
 <wire x1="99.06" y1="34.29" x2="100.654584375" y2="34.487584375" width="0" layer="19" extent="1-1"/>
@@
 <wire x1="35.955" y1="34.98" x2="39.445303125" y2="36.5125" width="0" layer="19" extent="1-16"/>
 <wire x1="2.22" y1="-6.35" x2="25.868" y2="22.362" width="0" layer="19" extent="1-1"/>
+<wire x1="-3.68" y1="-11.7" x2="2.22" y2="-6.35" width="0" layer="19" extent="1-1"/>
+<wire x1="-3.68" y1="-12.2" x2="-3.68" y2="-11.7" width="0" layer="19" extent="1-1"/>
+<wire x1="-3.68" y1="-13.2" x2="-3.68" y2="-12.2" width="0" layer="19" extent="1-1"/>
+<wire x1="-5.08" y1="-11.3" x2="-3.68" y2="-11.7" width="0" layer="19" extent="1-1"/>
+<wire x1="-5.58" y1="-11.3" x2="-5.08" y2="-11.3" width="0" layer="19" extent="1-1"/>
+<wire x1="-5.08" y1="-14.1" x2="-3.68" y2="-13.2" width="0" layer="19" extent="1-1"/>
+<wire x1="-6.48" y1="-13.7" x2="-5.08" y2="-14.1" width="0" layer="19" extent="1-1"/>
+<wire x1="-3.68" y1="-25.4" x2="-5.08" y2="-14.1" width="0" layer="19" extent="1-1"/>
+<wire x1="-3.68" y1="-31.75" x2="-3.68" y2="-25.4" width="0" layer="19" extent="1-1"/>
 </signal>
 <signal name="N$1">
@@
 </signal>
 <signal name="+5V">
-<contactref element="PTCFUSE" pad="2"/>
-<contactref element="U$1" pad="7"/>
-<contactref element="U$1" pad="2"/>
-<wire x1="81.554465625" y1="24.54309375" x2="81.56609375" y2="24.54309375" width="0.254" layer="1"/>
-<wire x1="81.56609375" y1="24.54309375" x2="82.677" y2="25.654" width="0.254" layer="1"/>
-<wire x1="82.677" y1="25.654" x2="82.677" y2="26.162" width="0.254" layer="1"/>
-<wire x1="82.677" y1="26.162" x2="80.391" y2="28.448" width="0.254" layer="1"/>
-<wire x1="80.391" y1="28.448" x2="79.802515625" y2="28.448" width="0.254" layer="1"/>
-<wire x1="79.802515625" y1="28.448" x2="78.7260375" y2="27.371521875" width="0.254" layer="1"/>
 <contactref element="C5" pad="1"/>
 <contactref element="C6" pad="+"/>
-<wire x1="65.027" y1="31.75" x2="67.19716875" y2="31.75" width="0.254" layer="1"/>
 <wire x1="67.19716875" y1="31.75" x2="68.41356875" y2="32.9664" width="0.254" layer="1"/>
 <wire x1="68.41356875" y1="32.9664" x2="70.1086" y2="32.9664" width="0.254" layer="1"/>
 <wire x1="70.1086" y1="32.9664" x2="72.595" y2="30.48" width="0.254" layer="1"/>
 <wire x1="80.33" y1="20.32" x2="80.33" y2="23.318628125" width="0.254" layer="1"/>
-<wire x1="80.33" y1="23.318628125" x2="81.554465625" y2="24.54309375" width="0.254" layer="1"/>
 <wire x1="72.595" y1="30.48" x2="74.93" y2="30.099" width="0.254" layer="1"/>
 <contactref element="Q2" pad="4"/>
 <contactref element="R5" pad="1"/>
 <contactref element="D11" pad="A"/>
-<wire x1="74.93" y1="30.099" x2="78.7260375" y2="27.371521875" width="0" layer="19" extent="1-1"/>
-<wire x1="4.445" y1="7.56" x2="65.027" y2="31.75" width="0" layer="19" extent="1-1"/>
+<wire x1="74.93" y1="30.099" x2="80.33" y2="23.318628125" width="0" layer="19" extent="1-1"/>
+<wire x1="4.445" y1="7.56" x2="67.19716875" y2="31.75" width="0" layer="19" extent="1-1"/>
 <wire x1="7.28" y1="-1.27" x2="4.445" y2="7.56" width="0" layer="19" extent="1-1"/>
 <wire x1="0.32" y1="-6.35" x2="7.28" y2="-1.27" width="0" layer="19" extent="1-1"/>
@@
 <contactref element="D11" pad="C"/>
 <contactref element="D12" pad="C"/>
+<contactref element="U2" pad="14"/>
+<contactref element="C21" pad="1"/>
+<contactref element="C22" pad="1"/>
+<contactref element="R8" pad="1"/>
 <wire x1="89.855" y1="30.48" x2="89.31114375" y2="30.57685625" width="0" layer="19" extent="1-16"/>
 <wire x1="73.787" y1="23.749" x2="70.805" y2="30.48" width="0" layer="19" extent="1-16"/>
 <wire x1="2.88" y1="-1.27" x2="45.405" y2="30.48" width="0" layer="19" extent="1-16"/>
-<wire x1="2.88" y1="-13.97" x2="2.88" y2="-1.27" width="0" layer="19" extent="1-1"/>
+<wire x1="-4.58" y1="-11.3" x2="2.88" y2="-1.27" width="0" layer="19" extent="1-1"/>
+<wire x1="2.88" y1="-13.97" x2="-4.58" y2="-11.3" width="0" layer="19" extent="1-1"/>
+<wire x1="-6.48" y1="-25.4" x2="-4.58" y2="-11.3" width="0" layer="19" extent="1-1"/>
+<wire x1="-6.48" y1="-31.75" x2="-6.48" y2="-25.4" width="0" layer="19" extent="1-1"/>
+<wire x1="-6.03" y1="-48.26" x2="-6.48" y2="-31.75" width="0" layer="19" extent="1-1"/>
 </signal>
 <signal name="N$6">
@@
 <wire x1="7.28" y1="-13.97" x2="4.445" y2="12.76" width="0" layer="19" extent="1-1"/>
 </signal>
+<signal name="SDA">
+<contactref element="U2" pad="4"/>
+<contactref element="R6" pad="2"/>
+<contactref element="U$1" pad="19"/>
+<wire x1="-6.48" y1="-13.2" x2="90.3225875" y2="26.24015" width="0" layer="19" extent="1-1"/>
+<wire x1="-4.13" y1="-38.1" x2="-6.48" y2="-13.2" width="0" layer="19" extent="1-1"/>
+</signal>
+<signal name="SCL">
+<contactref element="U2" pad="6"/>
+<contactref element="R7" pad="2"/>
+<contactref element="U$1" pad="18"/>
+<wire x1="-5.58" y1="-14.1" x2="89.756903125" y2="25.674465625" width="0" layer="19" extent="1-1"/>
+<wire x1="-4.13" y1="-43.18" x2="-5.58" y2="-14.1" width="0" layer="19" extent="1-1"/>
+</signal>
+<signal name="N$23">
+<contactref element="U2" pad="1"/>
+<contactref element="R6" pad="1"/>
+<contactref element="R7" pad="1"/>
+<wire x1="-6.03" y1="-38.1" x2="-6.03" y2="-43.18" width="0" layer="19" extent="1-1"/>
+<wire x1="-6.48" y1="-11.7" x2="-6.03" y2="-38.1" width="0" layer="19" extent="1-1"/>
+</signal>
+<signal name="N$18">
+<contactref element="U2" pad="8"/>
+<contactref element="R8" pad="2"/>
+<wire x1="-4.58" y1="-14.1" x2="-4.13" y2="-48.26" width="0" layer="19" extent="1-1"/>
+</signal>
+<signal name="ACCEL_INT1">
+<contactref element="U2" pad="11"/>
+<contactref element="U$1" pad="20"/>
+<wire x1="-3.68" y1="-12.7" x2="90.888275" y2="26.805834375" width="0" layer="19" extent="1-1"/>
+</signal>
+<signal name="ACCEL_INT2">
+<contactref element="U2" pad="9"/>
+<contactref element="U$1" pad="21"/>
+<wire x1="-3.68" y1="-13.7" x2="91.453959375" y2="27.371521875" width="0" layer="19" extent="1-1"/>
+</signal>
+<signal name="V_USB">
+<contactref element="PTCFUSE" pad="2"/>
+<contactref element="U$1" pad="7"/>
+<contactref element="U$1" pad="2"/>
+<wire x1="81.56609375" y1="24.54309375" x2="82.677" y2="25.654" width="0.254" layer="1"/>
+<wire x1="82.677" y1="25.654" x2="82.677" y2="26.162" width="0.254" layer="1"/>
+<wire x1="82.677" y1="26.162" x2="80.391" y2="28.448" width="0.254" layer="1"/>
+<wire x1="80.391" y1="28.448" x2="79.802515625" y2="28.448" width="0.254" layer="1"/>
+<wire x1="79.802515625" y1="28.448" x2="78.7260375" y2="27.371521875" width="0.254" layer="1"/>
+<wire x1="81.56609375" y1="24.54309375" x2="81.554465625" y2="24.54309375" width="0" layer="19" extent="1-1"/>
+<wire x1="65.027" y1="31.75" x2="78.7260375" y2="27.371521875" width="0" layer="19" extent="1-1"/>
+</signal>
 </signals>

Commit message: WIP
Parts:
- removed AREF: PTR1B1,27, testpad:B1,27
- removed C10, C11, C12, C13, C14, C15, C16, C17, C18, C7, C9: 0.1uF, microbuilder:0805
- removed D1, D10, D2, D3, D4, D5, D6, D7, D8, D9: WS2812B, SparkFun-LED:WS2812B
- removed D11, D12: (no value), eagle-ltspice:DIODE_SMB
- removed ISP: (no value), pinhead:2X03
- removed S3: (no value), SparkFun-Switches:SWITCH_SPST_SMD_A
- removed U1: CR2032-SNAPDRAGONCR2032, CR2032-SnapDragon:CR2032-SNAPDRAGON
- added AREF1: PTR1B1,27, testpad:B1,27
- added C23, C27: 1uF, microbuilder:0805
- added C24, C25, C26: 10uF, microbuilder:0805
- added CHG: Orange APT2012SECK, microbuilder:CHIPLED_0805
- added D13: (no value), adafruit:SOD-123
- added EN: (no value), microbuilder:SPDT_SMT_SSSS811101
- added IC1: MCP73831/OT, adafruit:SOT23-5L
- added POWER: (no value), adafruit:JST-PH-2-THM
- added Q1: 220mA/50V/3.5Ω, SparkFun-DiscreteSemi:SOT23-3
- added R10, R13, R17, R9: 10k, microbuilder:0805
- added R11, R14, R16: 100k, microbuilder:0805
- added R12: 1k, microbuilder:0805
- added U$10, U$11, U$12, U$13, U$4, U$5, U$6, U$7, U$8, U$9: APA1025050, jos-ph:APA102_5050
- added U3: 3.3V, SparkFun-IC-Power:SOT23-5
- Q2: value (none) -> 220mA/50V/3.5Ω; device transistor-power:SO-08 -> SparkFun-DiscreteSemi:SOT23-3
- moved Q2 211.5 mm to (-14.0, -200.7)
- moved R5 182.4 mm to (-15.2, -188.0)
Connections:
- removed net MISO: ISP.1, U$1.11
- removed net MOSI: ISP.4, U$1.10
- removed net N$20: D12.A, Q2.5, Q2.6, Q2.7, Q2.8
- removed net N$33: S3.1, U1.V+
- removed net N$4: C20.1, Q2.1, Q2.2, Q2.3, R3.1, U$2.5
- removed net SCK: ISP.3, U$1.9
- removed net VIN: C19.1, L1.1, S3.2, U$2.3, U$2.6
- new net +3V3: C19.1, C21.1, C22.1, C25.1, C27.1, L1.1, Q1.2, Q2.2, R10.1, R5.1, R8.1, U$1.14, U$1.24, U$1.34, U$1.44, U$2.3, U$2.6, U2.14, U3.5
- new net 5V: C20.1, Q1.3, Q2.3, R17.1, R3.1, R9.1, U$10.1, U$11.1, U$12.1, U$13.1, U$2.5, U$4.1, U$5.1, U$6.1, U$7.1, U$8.1, U$9.1
- new net C_HL: R17.2, U$4.5
- new net C_LL: Q2.1, R10.2
- new net D_HL: R9.2, U$1.40, U$4.4
- new net D_LL: Q1.1, R5.2, U$1.41
- new net EN: EN.B, R11.2, U3.3
- new net N$21: U$10.4, U$9.3
- new net N$22: U$10.5, U$9.2
- new net N$24: U$10.2, U$11.5
- new net N$25: U$10.3, U$11.4
- new net N$26: IC1.1, R12.2
- new net N$27: U$11.3, U$12.4
- new net N$28: CHG.C, R12.1
- new net N$29: U$11.2, U$12.5
- new net N$30: IC1.5, R13.1
- new net N$31: U$12.2, U$13.5
- new net N$35: U$12.3, U$13.4
- new net V_BATT: C26.1, D13.A, IC1.3, POWER.2, R16.2
- net +5V: no longer D11.A, Q2.4, R5.1
- net AREF: now also AREF1.TP, C23.1; no longer AREF.TP, C7.1
- net GND: now also C23.2, C24.2, C25.2, C26.2, C27.2, EN.A, IC1.2, POWER.1, R13.2, R14.1, U$10.6, U$11.6, U$12.6, U$13.6, U$4.6, U$5.6, U$6.6, U$7.6, U$8.6, U$9.6, U3.2; no longer C10.2, C11.2, C12.2, C13.2, C14.2, C15.2, C16.2, C17.2, C18.2, C7.2, C9.2, D1.3, D10.3, D2.3, D3.3, D4.3, D5.3, D6.3, D7.3, D8.3, D9.3, ISP.6, R5.2, U1.V-
- net N$10: now also U$5.3, U$6.4; no longer D3.2, D4.4
- net N$11: now also U$5.2, U$6.5; no longer D4.2, D5.4
- net N$12: now also U$6.3, U$7.4; no longer D5.2, D6.4
- net N$13: now also U$6.2, U$7.5; no longer D6.2, D7.4
- net N$14: now also U$7.3, U$8.4; no longer D7.2, D8.4
- net N$15: now also U$7.2, U$8.5; no longer D8.2, D9.4
- net N$16: now also U$8.3, U$9.4; no longer D10.4, D9.2
- net N$17: now also U$8.2, U$9.5; no longer D1.4
- net N$32: now also R14.2, R16.1
- net N$8: now also U$4.3, U$5.4; no longer D1.2, D2.4
- net N$9: now also U$4.2, U$5.5; no longer D2.2, D3.4
- net RST: no longer ISP.5
- net VCC: no longer C10.1, C11.1, C12.1, C13.1, C14.1, C15.1, C16.1, C17.1, C18.1, C21.1, C22.1, C9.1, D1.1, D10.1, D11.C, D12.C, D2.1, D3.1, D4.1, D5.1, D6.1, D7.1, D8.1, D9.1, ISP.2, R8.1, U$1.14, U$1.24, U$1.34, U$1.44, U2.14
- net V_USB: now also C24.1, CHG.A, D13.C, IC1.4, R11.1, U3.1
Routing:
- net VCC: track 230.0 -> 10.3 mm
- net MOSI: track 46.8 -> 0.00 mm, vias 1 -> 0
- net SCK: track 41.9 -> 0.00 mm, vias 1 -> 0
- net +3V3: track 0.00 -> 41.0 mm
- net MISO: track 40.5 -> 0.00 mm, vias 1 -> 0
- net GND: track 140.8 -> 107.2 mm
- net N$33: track 26.3 -> 0.00 mm
- net RST: track 92.9 -> 70.1 mm
- net VIN: track 15.2 -> 0.00 mm
- net N$4: track 7.57 -> 0.00 mm
- net 5V: track 0.00 -> 7.57 mm
- net N$15: track 6.46 -> 0.00 mm
- net N$13: track 6.46 -> 0.00 mm
- net N$12: track 6.46 -> 0.00 mm
- net N$10: track 6.46 -> 0.00 mm
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
Commit message: WIP
Parts:
- removed AREF1: PTR1B1,27, testpad:B1,27
- removed C19: 4.7uF, microbuilder:0805
- removed C20, C24, C25, C26: 10uF, microbuilder:0805
- removed C23, C27: 1uF, microbuilder:0805
- removed U$1: ATMEGA32U4-AU, adafruit:TQFP44
- added C10, C11, C14, C9: 10uF, rcl:C0603K
- added C12: 1uF, rcl:C0603K
- added C7: 18pF, rcl:C0603K
- added R18: 10k, microbuilder:0603
- added U$3: 32U4, SparkFun-IC-Microcontroller:QFN-44
- C1, C3, C4: device microbuilder:0805 -> rcl:C0603K
- C2: value 18pF -> 0.1uF; device microbuilder:0805 -> rcl:C0603K
- C21, C22: device rcl:C1206 -> rcl:C0603K
- C5: value 0.1uF -> 1uF; device microbuilder:0805 -> rcl:C0603K
- C6: device microbuilder:EIA3216-18/A-W -> microbuilder:EIA3216-18/A-R
- C8: value 1uF -> 4.7uF; device microbuilder:0805 -> rcl:C0603K
- CHG, LED13: device microbuilder:CHIPLED_0805 -> microbuilder:CHIPLED_0603
- R1, R10, R11, R12, R13, R14, R15, R16, R17, R2, R3, R4, R5, R6, R7, R8, R9: device microbuilder:0805 -> microbuilder:0603
- moved R17 253.9 mm to (40.6, 34.3), turned to 90 degrees
- moved R10 250.1 mm to (45.7, 34.3), turned to 270 degrees
- moved Q2 241.8 mm to (43.2, 34.3), turned to 90 degrees
- moved R9 237.8 mm to (40.6, 38.1), turned to 270 degrees
- moved U$13 235.9 mm to (96.5, 36.8), flipped to the bottom, turned to 90 degrees
- moved R5 234.1 mm to (45.7, 38.1), turned to 270 degrees
- moved U$12 226.8 mm to (91.4, 36.8), flipped to the bottom, turned to 90 degrees
- moved Q1 223.6 mm to (43.2, 38.1), turned to 90 degrees
- moved U$11 217.8 mm to (86.4, 36.8), flipped to the bottom, turned to 90 degrees
- moved U$10 208.8 mm to (81.3, 36.8), flipped to the bottom, turned to 90 degrees
- moved U$9 199.8 mm to (76.2, 36.8), flipped to the bottom, turned to 90 degrees
- moved U$8 190.8 mm to (71.1, 36.8), flipped to the bottom, turned to 90 degrees
- moved U$7 181.8 mm to (66.0, 36.8), flipped to the bottom, turned to 90 degrees
- moved U$6 172.9 mm to (61.0, 36.8), flipped to the bottom, turned to 90 degrees
- moved U$5 164.0 mm to (55.9, 36.8), flipped to the bottom, turned to 90 degrees
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Connections:
- removed net +5V: C5.1, C6.+
- removed net ACCEL_INT2: U$1.21, U2.9
- removed net AREF: AREF1.TP, C23.1, U$1.42
- removed net C_HL: R17.2, U$4.5
- removed net C_LL: Q2.1, R10.2
- removed net D_HL: R9.2, U$1.40, U$4.4
- removed net D_LL: Q1.1, R5.2, U$1.41
- removed net N$23: R6.1, R7.1, U2.1
- removed net N$34: C8.1, U$1.6
- removed net PE6: S1.1, U$1.1
- removed net VCC: C3.1, C4.1
- new net HV1: Q1.3, R9.1, U$4.4
- new net HV2: Q2.3, R17.1, U$4.5
- new net LV1: Q1.2, R5.1, U$3.40
- new net LV2: Q2.2, R10.1, U$3.41
- new net N$4: R18.1, U2.7
- new net PF6: S1.1, U$3.37
- net +3V3: now also C11.1, C12.1, C2.2, C3.2, C5.2, C8.1, Q1.1, Q2.1, R10.2, R5.2, R6.1, R7.1, U$3.24, U$3.44, U2.1; no longer C19.1, C25.1, C27.1, Q1.2, Q2.2, R10.1, R5.1, U$1.14, U$1.24, U$1.34, U$1.44
- net 5V: now also C9.1, R17.2, R9.2; no longer C20.1, Q1.3, Q2.3, R17.1, R9.1
- net ACCEL_INT1: now also U$3.29; no longer U$1.20
- net GND: now also C10.2, C11.2, C12.2, C14.2, C3.1, C4.1, C5.1, C7.1, C9.2, R18.2; no longer C19.2, C20.2, C23.2, C24.2, C25.2, C26.2, C27.2, C3.2, C4.2, C5.2, U$1.15, U$1.23, U$1.35, U$1.43, U$1.5, U2.7
- net N$6: now also C7.2, U$3.16; no longer C2.2, U$1.16
- net N$7: now also U$3.17; no longer U$1.17
- net PB0: now also U$3.8; no longer U$1.8
- net PD5: now also U$3.22; no longer U$1.22
- net RST: now also U$3.13; no longer U$1.13
- net SCL: now also U$3.18; no longer U$1.18
- net SDA: now also U$3.19; no longer U$1.19
- net USB_D+: now also U$3.4; no longer U$1.4
- net USB_D-: now also U$3.3; no longer U$1.3
- net V_BATT: now also C14.1; no longer C26.1
- net V_USB: now also C10.1, C4.2, C6.+, U$3.7; no longer C24.1, U$1.2, U$1.7
Routing:
- net PB0: track 87.9 -> 0.00 mm, vias 2 -> 0
- net 5V: track 7.57 -> 78.2 mm, vias 0 -> 1
- net RST: track 70.1 -> 0.00 mm, vias 1 -> 0
- net PE6: track 63.2 -> 0.00 mm
- net PD5: track 27.8 -> 0.00 mm, vias 2 -> 0
- net N$34: track 21.8 -> 0.00 mm, vias 2 -> 0
- net LV1: track 0.00 -> 21.1 mm
- net HV2: track 0.00 -> 16.7 mm, vias 0 -> 1
- net HV1: track 0.00 -> 13.7 mm, vias 0 -> 1
- net AREF: track 13.1 -> 0.00 mm
- net +5V: track 12.3 -> 0.00 mm
- net SCL: track 0.00 -> 10.7 mm
- net VCC: track 10.3 -> 0.00 mm
- net N$7: track 14.5 -> 5.95 mm
- net N$16: track 0.00 -> 6.95 mm
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Other:
- board size 98.7 x 22.9 mm -> 89.8 x 20.3 mm
- board text removed: "GND"
- board text removed: "MISO"
- board text removed: "MOSI"
- board text removed: "SCK"
- board text removed: "VCC"
