File: POIstick/POIstick2.sch (EAGLE design)
At the start: 39 parts, among them U1 CR2032-SNAPDRAGONCR2032, X1 8MHz

Commit message: initial V2
Parts:
- removed F2: (no value), adafruit:PTCFUSE-1206
- added AREF: PTR1B1,27, testpad:PTR1B1,27
- added C8: 1uF, microbuilder:CAP_CERAMIC0805
- added LED13: APT2012SECK, microbuilder:LED0805
- added PTCFUSE: 500mA, microbuilder:PTC1206
- added R15: 47, microbuilder:RESISTOR0805
- added S1: MOMENTARY-SWITCH-SPST-SMD-12MM, SparkFun-Switches:MOMENTARY-SWITCH-SPST-SMD-12MM
- added S3: (no value), SparkFun-Switches:SWITCH-SPDT-SMD-RIGHT-ANGLE
- added SW1, SW2: 431151015826, Wurth_Elektronik_Electromechanic_Switchs_rev15b:431151015826
- C1, C2, C4, C5: device rcl:C-EUC1206 -> microbuilder:CAP_CERAMIC0805
- C3: value (none) -> 0.1uF; device rcl:C-EUC1206 -> microbuilder:CAP_CERAMIC0805
- C6: value 0.1uF -> 10uF; device rcl:C-EUC1206 -> microbuilder:CAP_TANTALUMA/3216_WAVE
- C7: value 10uF -> 0.1uF; device resistor:CPOL-USCT3216 -> microbuilder:CAP_CERAMIC0805
- LED1: value (none) -> Orange APT2012SECK; device adafruit:LEDCHIPLED_0805 -> microbuilder:LED0805
- LED10, LED11, LED12, LED2, LED3, LED4, LED5, LED6, LED7, LED8, LED9: value (none) -> APT2012SECK; device adafruit:LEDCHIPLED_0805 -> microbuilder:LED0805
- R1, R2: device adafruit:R-US_R0805 -> microbuilder:RESISTOR0805
- R10, R11, R12, R13, R14, R3, R4, R5, R6, R7, R8, R9: value 22 -> 47; device adafruit:R-US_R0805 -> microbuilder:RESISTOR0805
- X1: value 8MHz -> 2MHz
Connections:
- removed net +3V3: C3.2, U$1.UCAP
- new net N$32: LED13.C, R15.1
- new net N$33: S3.O, U1.V+
- new net N$34: C8.P$1, U$1.UCAP
- new net PB0: SW2.2, U$1.PB0(SS)
- new net PD5: LED13.A, U$1.PD5(XCK/CTS)
- new net PE6: S1.1, U$1.PE6(INT.6/AIN0)
- net +5V: now also C5.P$1, C6.+, PTCFUSE.2; no longer C6.2, C7.+, F2.2
- net AREF: now also AREF.TP, C7.P$1
- net GND: now also C1.P$1, C2.P$1, C3.P$2, C4.P$2, C5.P$2, C6.-, C7.P$2, C8.P$2, R15.2, S1.2, SW1.2, SW2.1, U1.V-; no longer C1.1, C2.1, C3.1, C4.1, C5.1, C6.1, C7.-
- net N$5: now also PTCFUSE.1; no longer F2.1
- net N$6: now also C2.P$2; no longer C2.2
- net N$7: now also C1.P$2; no longer C1.2
- net RST: now also SW1.1
- net VCC: now also C3.P$1, C4.P$1, S3.P; no longer C4.2, C5.2
Other:
- note removed: "BHSD-2032-SMCT-ND"
- moved on the sheet: C3, C4, C5, ISP, U1

Commit message: WIP
Parts:
- removed LED1: Orange APT2012SECK, microbuilder:LED0805
- removed LED10, LED11, LED12, LED2, LED3, LED4, LED5, LED6, LED7, LED8, LED9: APT2012SECK, microbuilder:LED0805
- removed R10, R11, R12, R13, R14, R3, R4, R5, R6, R7, R8, R9: 47, microbuilder:RESISTOR0805
- added C10, C11, C12, C13, C14, C15, C16, C17, C18, C9: 0.1uF, microbuilder:CAP_CERAMIC0805
- added D1, D10, D2, D3, D4, D5, D6, D7, D8, D9: WS2812B, SparkFun-LED:WS2812B
- ISP: SPICEPREFIX (none) -> X
Connections:
- removed net N$20: LED7.C, R9.1
- removed net N$21: LED7.A, U$1.PE2(!HWB)
- removed net N$22: LED8.C, R10.1
- removed net N$23: LED8.A, U$1.PC7(ICP3/CLK0/OC4A)
- removed net N$24: LED9.C, R11.1
- removed net N$25: LED9.A, U$1.PC6(OC3A/!OC4A)
- removed net N$26: LED10.C, R12.1
- removed net N$27: LED10.A, U$1.PB6(OC1B/OC4B/ADC13)
- removed net N$28: LED11.C, R13.1
- removed net N$29: LED11.A, U$1.PB5(OC1A/ADC12/!OC4B)
- removed net N$30: LED12.C, R14.1
- removed net N$31: LED12.A, U$1.PB4(ADC11)
- net GND: now also C10.P$2, C11.P$2, C12.P$2, C13.P$2, C14.P$2, C15.P$2, C16.P$2, C17.P$2, C18.P$2, C9.P$2, D1.VSS, D10.VSS, D2.VSS, D3.VSS, D4.VSS, D5.VSS, D6.VSS, D7.VSS, D8.VSS, D9.VSS; no longer R10.2, R11.2, R12.2, R13.2, R14.2, R3.2, R4.2, R5.2, R6.2, R7.2, R8.2, R9.2
- net N$10: now also D3.DO, D4.DI; no longer LED2.C, R4.1
- net N$11: now also D4.DO, D5.DI; no longer LED1.A, U$1.PF7(ADC7(TDI)
- net N$12: now also D5.DO, D6.DI; no longer LED3.C, R5.1
- net N$13: now also D6.DO, D7.DI; no longer LED3.A, U$1.PF5(ADC5/TMS)
- net N$14: now also D7.DO, D8.DI; no longer LED4.C, R6.1
- net N$15: now also D8.DO, D9.DI; no longer LED4.A, U$1.PF4(ADC4/TCK)
- net N$16: now also D10.DI, D9.DO; no longer LED5.C, R7.1
- net N$17: now also D1.DI; no longer LED5.A, U$1.PF1(ADC1)
- net N$18: now also R1.2; no longer LED6.C, R8.1
- net N$19: now also R2.2; no longer LED6.A, U$1.PF0(ADC0)
- net N$3: now also U$1.D-; no longer R1.2, U$1.D+
- net N$4: now also U$1.D+; no longer R2.2, U$1.D-
- net N$8: now also D1.DO, D2.DI; no longer LED1.C, R3.1
- net N$9: now also D2.DO, D3.DI; no longer LED2.A, U$1.PF6(ADC6/TDO)
- net VCC: now also C10.P$1, C11.P$1, C12.P$1, C13.P$1, C14.P$1, C15.P$1, C16.P$1, C17.P$1, C18.P$1, C9.P$1, D1.VDD, D10.VDD, D2.VDD, D3.VDD, D4.VDD, D5.VDD, D6.VDD, D7.VDD, D8.VDD, D9.VDD
Other:
- note added: "Control switches"
- note added: "Control/activity LED"
- note added: "ISP"
- note added: "LED Array/Line"
- note added: "MCU"
- note added: "Power"
- note added: "USB"
- moved on the sheet: C1, C2, C3, C4, C5, C6, CN1, ISP, LED13, PTCFUSE, R1, R15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

Commit message: WIP
Parts:
- added C19: 4.7uF, microbuilder:CAP_CERAMIC0805
- added C20: 10uF, microbuilder:CAP_CERAMIC0805
- added L1: 4.7uH, WE-TPC:WE-TPC-744031004_3816
- added R3: 976K, microbuilder:RESISTOR0805
- added R4: 309K, microbuilder:RESISTOR0805
- added U$2: MCP1623/24, MCP1623:MCP1623/24
- X1: value 2MHz -> 8MHz
Connections:
- removed net N$18: R1.2
- removed net N$4: U$1.D+
- new net USB_D+: R1.2, U$1.D+
- new net USB_D-: R2.2, U$1.D-
- new net VIN: C19.P$1, L1.1, S3.P, U$2.EN, U$2.VIN
- net GND: now also C19.P$2, C20.P$2, R4.2, U$2.GND
- net N$19: now also L1.2, U$2.SW; no longer R2.2
- net N$3: now also R3.2, R4.1, U$2.VFB; no longer U$1.D-
- net VCC: now also C20.P$1, R3.1, U$2.VOUT; no longer S3.P
Other:
- note added: "AREF"
- moved on the sheet: AREF, C1, C10, C11, C12, C13, C14, C15, C16, C17, C18, C2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

Commit message: WIP
Parts:
- added D11, D12: (no value), eagle-ltspice:SCHOTTKY-DIODE
- added Q2: (no value), transistor-power:P-MOSFET-SO8
- added R5: 10k, microbuilder:RESISTOR0805
Connections:
- new net N$20: D12.C, Q2.D
- new net N$4: C20.P$1, Q2.S, R3.1, U$2.VOUT
- net +5V: now also D11.C, Q2.G, R5.1
- net GND: now also R5.2
- net VCC: now also D11.A, D12.A; no longer C20.P$1, R3.1, U$2.VOUT
Other:
- moved on the sheet: C19, C20, C3, C4, C5, C6, L1, R3, R4, S3, U$2, U1

Commit message: WIP
Parts:
- added C21: 0.1uF, rcl:C-EUC1206
- added C22: 10uF, rcl:C-EUC1206
- added R6, R7, R8: 10k, microbuilder:RESISTOR0805
- added U2: LIS3DH, SparkFun-Sensors:LIS3DH
Connections:
- new net ACCEL_INT1: U$1.PD2(INT2/RXD1), U2.INT1
- new net ACCEL_INT2: U$1.PD3(INT3/TXD1), U2.INT2
- new net N$18: R8.2, U2.!CS!/MODE
- new net N$23: R6.1, R7.1, U2.VDDIO
- new net SCL: R7.2, U$1.PD0(INT0/OC0B/SCL), U2.SDA/SDI
- new net SDA: R6.2, U$1.PD1(INT1/SDA), U2.SCL/SPC
- new net V_USB: PTCFUSE.2, U$1.UVCC, U$1.VBUS
- net +5V: no longer PTCFUSE.2, U$1.UVCC, U$1.VBUS
- net GND: now also C21.2, C22.2, U2.ADC1, U2.ADC2, U2.ADC3, U2.GND@12, U2.GND@5, U2.RES, U2.SA0/SDO
- net VCC: now also C21.1, C22.1, R8.1, U2.VDD
Other:
- note added: "Accelerometer"
- moved on the sheet: C1, C2, C8, U$1, X1

Commit message: WIP
Parts:
- removed AREF: PTR1B1,27, testpad:PTR1B1,27
- removed C10, C11, C12, C13, C14, C15, C16, C17, C18, C7, C9: 0.1uF, microbuilder:CAP_CERAMIC0805
- removed D1, D10, D2, D3, D4, D5, D6, D7, D8, D9: WS2812B, SparkFun-LED:WS2812B
- removed D11, D12: (no value), eagle-ltspice:SCHOTTKY-DIODE
- removed ISP: (no value), pinhead:PINHD-2X3
- removed S3: (no value), SparkFun-Switches:SWITCH-SPDT-SMD-RIGHT-ANGLE
- removed U1: CR2032-SNAPDRAGONCR2032, CR2032-SnapDragon:CR2032-SNAPDRAGONCR2032
- added AREF1: PTR1B1,27, testpad:PTR1B1,27
- added C23, C27: 1uF, microbuilder:CAP_CERAMIC0805
- added C24, C25, C26: 10uF, microbuilder:CAP_CERAMIC0805
- added CHG: Orange APT2012SECK, microbuilder:LED0805
- added D13: (no value), adafruit:DIODESOD-123
- added EN: (no value), microbuilder:SWITCH_SPDT
- added IC1: MCP73831/OT, adafruit:MCP73831/OT
- added POWER: (no value), adafruit:JST_2PIN-THM
- added Q1: 220mA/50V/3.5Ω, SparkFun-DiscreteSemi:MOSFET-NCH-BSS138
- added R10, R13, R17, R9: 10k, microbuilder:RESISTOR0805
- added R11, R14, R16: 100k, microbuilder:RESISTOR0805
- added R12: 1k, microbuilder:RESISTOR0805
- added U$10, U$11, U$12, U$13, U$4, U$5, U$6, U$7, U$8, U$9: APA1025050, jos-ph:APA1025050
- added U3: 3.3V, SparkFun-IC-Power:V_REG_AP2112K-3.3V
- Q2: value (none) -> 220mA/50V/3.5Ω; device transistor-power:P-MOSFET-SO8 -> SparkFun-DiscreteSemi:MOSFET-NCH-BSS138
Connections:
- removed net MISO: ISP.1, U$1.PB3(PDO/MISO)
- removed net MOSI: ISP.4, U$1.PB2(PDI/MOSI)
- removed net N$20: D12.C, Q2.D
- removed net N$33: S3.O, U1.V+
- removed net N$4: C20.P$1, Q2.S, R3.1, U$2.VOUT
- removed net SCK: ISP.3, U$1.PB1(SCK)
- removed net VIN: C19.P$1, L1.1, S3.P, U$2.EN, U$2.VIN
- new net +3V3: C19.P$1, C21.1, C22.1, C25.P$1, C27.P$1, L1.1, Q1.S, Q2.S, R10.1, R5.1, R8.1, U$1.AVCC, U$1.AVCC1, U$1.VCC, U$1.VCC1, U$2.EN, U$2.VIN, U2.VDD, U3.OUT
- new net 5V: C20.P$1, Q1.D, Q2.D, R17.1, R3.1, R9.1, U$10.VCC, U$11.VCC, U$12.VCC, U$13.VCC, U$2.VOUT, U$4.VCC, U$5.VCC, U$6.VCC, U$7.VCC, U$8.VCC, U$9.VCC
- new net C_HL: R17.2, U$4.CI
- new net C_LL: Q2.G, R10.2
- new net D_HL: R9.2, U$1.PF1(ADC1), U$4.DI
- new net D_LL: Q1.G, R5.2, U$1.PF0(ADC0)
- new net EN: EN.P, R11.2, U3.EN
- new net N$21: U$10.DI, U$9.DO
- new net N$22: U$10.CI, U$9.CO
- new net N$24: U$10.CO, U$11.CI
- new net N$25: U$10.DO, U$11.DI
- new net N$26: IC1.STAT, R12.2
- new net N$27: U$11.DO, U$12.DI
- new net N$28: CHG.C, R12.1
- new net N$29: U$11.CO, U$12.CI
- new net N$30: IC1.PROG, R13.1
- new net N$31: U$12.CO, U$13.CI
- new net N$35: U$12.DO, U$13.DI
- new net V_BATT: C26.P$1, D13.A, IC1.VBAT, POWER.1, R16.2
- net +5V: no longer D11.C, Q2.G, R5.1
- net AREF: now also AREF1.TP, C23.P$1; no longer AREF.TP, C7.P$1
- net GND: now also C23.P$2, C24.P$2, C25.P$2, C26.P$2, C27.P$2, EN.O, IC1.VSS, POWER.2, R13.2, R14.1, U$10.GND, U$11.GND, U$12.GND, U$13.GND, U$4.GND, U$5.GND, U$6.GND, U$7.GND, U$8.GND, U$9.GND, U3.GND; no longer C10.P$2, C11.P$2, C12.P$2, C13.P$2, C14.P$2, C15.P$2, C16.P$2, C17.P$2, C18.P$2, C7.P$2, C9.P$2, D1.VSS, D10.VSS, D2.VSS, D3.VSS, D4.VSS, D5.VSS, D6.VSS, D7.VSS, D8.VSS, D9.VSS, ISP.6, R5.2, U1.V-
- net N$10: now also U$5.DO, U$6.DI; no longer D3.DO, D4.DI
- net N$11: now also U$5.CO, U$6.CI; no longer D4.DO, D5.DI
- net N$12: now also U$6.DO, U$7.DI; no longer D5.DO, D6.DI
- net N$13: now also U$6.CO, U$7.CI; no longer D6.DO, D7.DI
- net N$14: now also U$7.DO, U$8.DI; no longer D7.DO, D8.DI
- net N$15: now also U$7.CO, U$8.CI; no longer D8.DO, D9.DI
- net N$16: now also U$8.DO, U$9.DI; no longer D10.DI, D9.DO
- net N$17: now also U$8.CO, U$9.CI; no longer D1.DI
- net N$32: now also R14.2, R16.1
- net N$8: now also U$4.DO, U$5.DI; no longer D1.DO, D2.DI
- net N$9: now also U$4.CO, U$5.CI; no longer D2.DO, D3.DI
- net RST: no longer ISP.5
- net VCC: no longer C10.P$1, C11.P$1, C12.P$1, C13.P$1, C14.P$1, C15.P$1, C16.P$1, C17.P$1, C18.P$1, C21.1, C22.1, C9.P$1, D1.VDD, D10.VDD, D11.A, D12.A, D2.VDD, D3.VDD, D4.VDD, D5.VDD, D6.VDD, D7.VDD, D8.VDD, D9.VDD, ISP.2, R8.1, U$1.AVCC, U$1.AVCC1, U$1.VCC, U$1.VCC1, U2.VDD
- net V_USB: now also C24.P$1, CHG.A, D13.C, IC1.VDD, R11.1, U3.IN
Other:
- note added: "Charge + Measure"
- note added: "Level Shifting"
- note added: "Power + Step-Down Regulator"
- note added: "Step-Up 3V3 -> 5V"
- note removed: "AREF"
- note removed: "ISP"
- note removed: "Power"
- moved on the sheet: C1, C19, C2, C20, C21, C22, C3, C4, C5, C6, C8, CN1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

Commit message: WIP
Parts:
- removed AREF1: PTR1B1,27, testpad:PTR1B1,27
- removed C19: 4.7uF, microbuilder:CAP_CERAMIC0805
- removed C20, C24, C25, C26: 10uF, microbuilder:CAP_CERAMIC0805
- removed C23, C27: 1uF, microbuilder:CAP_CERAMIC0805
- removed U$1: ATMEGA32U4-AU, adafruit:ATMEGA32U4-AU
- added C10, C11, C14, C9: 10uF, rcl:C-EUC0603K
- added C12: 1uF, rcl:C-EUC0603K
- added C7: 18pF, rcl:C-EUC0603K
- added R18: 10k, microbuilder:RESISTOR0603
- added U$3: 32U4, SparkFun-IC-Microcontroller:ATMEGA32U4QFN
- C1, C3, C4: device microbuilder:CAP_CERAMIC0805 -> rcl:C-EUC0603K
- C2: value 18pF -> 0.1uF; device microbuilder:CAP_CERAMIC0805 -> rcl:C-EUC0603K
- C21, C22: device rcl:C-EUC1206 -> rcl:C-EUC0603K
- C5: value 0.1uF -> 1uF; device microbuilder:CAP_CERAMIC0805 -> rcl:C-EUC0603K
- C6: device microbuilder:CAP_TANTALUMA/3216_WAVE -> microbuilder:CAP_TANTALUMA/3216_REFLOW
- C8: value 1uF -> 4.7uF; device microbuilder:CAP_CERAMIC0805 -> rcl:C-EUC0603K
- CHG, LED13: device microbuilder:LED0805 -> microbuilder:LED0603
- R1, R10, R11, R12, R13, R14, R15, R16, R17, R2, R3, R4, R5, R6, R7, R8, R9: device microbuilder:RESISTOR0805 -> microbuilder:RESISTOR0603
Connections:
- removed net +5V: C5.P$1, C6.+
- removed net ACCEL_INT2: U$1.PD3(INT3/TXD1), U2.INT2
- removed net AREF: AREF1.TP, C23.P$1, U$1.AREF
- removed net C_HL: R17.2, U$4.CI
- removed net C_LL: Q2.G, R10.2
- removed net D_HL: R9.2, U$1.PF1(ADC1), U$4.DI
- removed net D_LL: Q1.G, R5.2, U$1.PF0(ADC0)
- removed net N$23: R6.1, R7.1, U2.VDDIO
- removed net N$34: C8.P$1, U$1.UCAP
- removed net PE6: S1.1, U$1.PE6(INT.6/AIN0)
- removed net VCC: C3.P$1, C4.P$1
- new net HV1: Q1.D, R9.1, U$4.DI
- new net HV2: Q2.D, R17.1, U$4.CI
- new net LV1: Q1.S, R5.1, U$3.PF1(ADC1)
- new net LV2: Q2.S, R10.1, U$3.PF0(ADC0)
- new net N$4: R18.1, U2.SA0/SDO
- new net PF6: S1.1, U$3.PF6(ADC6)
- net +3V3: now also C11.1, C12.1, C2.2, C3.2, C5.2, C8.1, Q1.G, Q2.G, R10.2, R5.2, R6.1, R7.1, U$3.AVCC@24, U$3.AVCC@44, U2.VDDIO; no longer C19.P$1, C25.P$1, C27.P$1, Q1.S, Q2.S, R10.1, R5.1, U$1.AVCC, U$1.AVCC1, U$1.VCC, U$1.VCC1
- net 5V: now also C9.1, R17.2, R9.2; no longer C20.P$1, Q1.D, Q2.D, R17.1, R9.1
- net ACCEL_INT1: now also U$3.PB5(ADC12); no longer U$1.PD2(INT2/RXD1)
- net GND: now also C1.1, C10.2, C11.2, C12.2, C14.2, C2.1, C3.1, C4.1, C5.1, C7.1, C8.2, C9.2, R18.2; no longer C1.P$1, C19.P$2, C2.P$1, C20.P$2, C23.P$2, C24.P$2, C25.P$2, C26.P$2, C27.P$2, C3.P$2, C4.P$2, C5.P$2, C8.P$2, U$1.GND, U$1.GND1, U$1.GND2, U$1.GND3, U$1.UGND, U2.SA0/SDO
- net N$6: now also C7.2, U$3.XTAL2; no longer C2.P$2, U$1.XTAL2
- net N$7: now also C1.2, U$3.XTAL1; no longer C1.P$2, U$1.XTAL1
- net PB0: now also U$3.PB0(SS); no longer U$1.PB0(SS)
- net PD5: now also U$3.PD5; no longer U$1.PD5(XCK/CTS)
- net RST: now also U$3.!RESET; no longer U$1./RESET
- net SCL: now also U$3.PD0(SCL); no longer U$1.PD0(INT0/OC0B/SCL)
- net SDA: now also U$3.PD1(SDA); no longer U$1.PD1(INT1/SDA)
- net USB_D+: now also U$3.D+; no longer U$1.D+
- net USB_D-: now also U$3.D-; no longer U$1.D-
- net V_BATT: now also C14.1; no longer C26.P$1
- net V_USB: now also C10.1, C4.2, C6.+, U$3.VBUS; no longer C24.P$1, U$1.UVCC, U$1.VBUS
Other:
- moved on the sheet: C2, C3, C4, C5, C6, C8, Q1, Q2, R10, R17, R9
